File: Schematics/SiC_Single_Phase_Inverter.kicad_pcb (KiCad board)
At the start: 2 copper layers, 204.5 x 65.2 mm, 163 parts, among them IC1 F280049CPMSR, IC2 TPD2EUSB30ADRTR, IC3 CP2102N-A02-GQFN24R, J1 23AH8786-Red, J10 464369202, J11 464379202, J12 43650-0418, J13 464369202, J14 464379202, J15 43650-0418, J16 464369202, J17 43650-0418, J18 43650-0418, J19 FTSH-105-01-LM-D-K, J2 23AH8785-Black, J20 43650-0418, J21 43650-0418, J22 43045-1212, J23 43045-1212, J24 1051330011, J3 23AH8786-Red, J4 23AH8785-Black, J5 464379202, J6 464369202, J7 464379202, J8 464369202, J9 464379202, Q1 STB10NK60ZT4, Q2 C3M0025065K, Q3 C3M0025065K, Q4 C3M0025065K, Q5 C3M0025065K, Q6 STB10NK60ZT4, U1 UCC21710QDWRQ1, U2 UCC21710QDWRQ1, U3 UCC21710QDWRQ1, U4 UCC21710QDWRQ1, U5 TR05S3V3, Y1 ABM8-20.000MHZ-B2-T

Commit message: [Milestone Compelted Controller and USB]
- Added Test Points
- Completed USB circuit to Controller
- Wired up Controller
- Added Connectors to Power Subsheet and 12pin from cotnroller to Full
  Bridge
- Added 3d models for USB compoents
- General fixes to subsheets
Parts:
- added J25: 43650-0418, SiC_Inverter:436500418, F.Cu at (503.9, 92.2)
- added J26: 1051330011, SiC_Inverter:105133-0011, F.Cu at (498.4, 127.7)
- added TP1: 5277, SiC_Inverter:5277, F.Cu at (392.4, 164.8)
- added TP10: 5277, SiC_Inverter:5277, F.Cu at (368.8, 156.7)
- added TP11: 5277, SiC_Inverter:5277, F.Cu at (392.4, 72.2)
- added TP12: 5277, SiC_Inverter:5277, F.Cu at (392.4, 78.4)
- added TP13: 5277, SiC_Inverter:5277, F.Cu at (392.4, 84.7)
- added TP14: 5277, SiC_Inverter:5277, F.Cu at (392.4, 91.0)
- added TP15: 5277, SiC_Inverter:5277, F.Cu at (392.4, 97.2)
- added TP16: 5277, SiC_Inverter:5277, F.Cu at (392.4, 103.5)
- added TP17: 5277, SiC_Inverter:5277, F.Cu at (398.6, 72.2)
- added TP18: 5277, SiC_Inverter:5277, F.Cu at (398.6, 78.4)
- added TP19: 5277, SiC_Inverter:5277, F.Cu at (398.6, 84.7)
- added TP2: 5281, SiC_Inverter:5281, F.Cu at (392.4, 171.0)
- added TP20: 5277, SiC_Inverter:5277, F.Cu at (398.6, 91.0)
- added TP21: 5277, SiC_Inverter:5277, F.Cu at (398.6, 97.2)
- added TP22: 5277, SiC_Inverter:5277, F.Cu at (398.6, 103.5)
- added TP23: 5277, SiC_Inverter:5277, F.Cu at (404.9, 72.2)
- added TP24: 5277, SiC_Inverter:5277, F.Cu at (404.9, 78.4)
- added TP25: 5277, SiC_Inverter:5277, F.Cu at (404.9, 84.7)
- added TP26: 5277, SiC_Inverter:5277, F.Cu at (404.9, 91.0)
- added TP27: 5277, SiC_Inverter:5277, F.Cu at (404.9, 97.2)
- added TP28: 5277, SiC_Inverter:5277, F.Cu at (404.9, 103.5)
- added TP29: 5281, SiC_Inverter:5281, F.Cu at (411.2, 72.2)
- added TP3: 5277, SiC_Inverter:5277, F.Cu at (392.4, 177.3)
- added TP30: 5281, SiC_Inverter:5281, F.Cu at (411.2, 78.4)
- added TP31: 5277, SiC_Inverter:5277, F.Cu at (411.2, 84.7)
- added TP32: 5281, SiC_Inverter:5281, F.Cu at (411.2, 91.0)
- added TP33: 5277, SiC_Inverter:5277, F.Cu at (343.0, 195.3)
- added TP34: 5277, SiC_Inverter:5277, F.Cu at (343.0, 201.6)
- added TP35: 5277, SiC_Inverter:5277, F.Cu at (304.1, 195.3)
- added TP36: 5277, SiC_Inverter:5277, F.Cu at (304.1, 201.6)
- added TP37: 5277, SiC_Inverter:5277, F.Cu at (474.6, 142.5)
- added TP38: 5277, SiC_Inverter:5277, F.Cu at (474.6, 148.7)
- added TP39: 5277, SiC_Inverter:5277, F.Cu at (474.6, 155.0)
- added TP4: 5281, SiC_Inverter:5281, F.Cu at (392.4, 183.6)
- added TP40: 5277, SiC_Inverter:5277, F.Cu at (480.9, 142.5)
- added TP41: 5277, SiC_Inverter:5277, F.Cu at (480.9, 148.7)
- added TP42: 5277, SiC_Inverter:5277, F.Cu at (480.9, 155.0)
- added TP43: 5281, SiC_Inverter:5281, F.Cu at (487.2, 142.5)
- added TP44: 5277, SiC_Inverter:5277, F.Cu at (487.2, 148.7)
- added TP45: 5281, SiC_Inverter:5281, F.Cu at (487.2, 155.0)
- added TP46: 5277, SiC_Inverter:5277, F.Cu at (466.0, 177.8)
- added TP47: 5281, SiC_Inverter:5281, F.Cu at (466.0, 184.1)
- added TP48: 5281, SiC_Inverter:5281, F.Cu at (492.8, 99.6)
- added TP49: 5277, SiC_Inverter:5277, F.Cu at (492.8, 105.9)
- added TP5: 5277, SiC_Inverter:5277, F.Cu at (447.7, 12.1)
- added TP50: 5281, SiC_Inverter:5281, F.Cu at (499.1, 99.6)
- added TP51: 5277, SiC_Inverter:5277, F.Cu at (499.1, 105.9)
- added TP52: 5281, SiC_Inverter:5281, F.Cu at (505.4, 99.6)
- added TP53: 5277, SiC_Inverter:5277, F.Cu at (505.4, 105.9)
- added TP6: 5281, SiC_Inverter:5281, F.Cu at (447.7, 18.3)
- added TP7: 5277, SiC_Inverter:5277, F.Cu at (464.2, 49.3)
- added TP8: 5281, SiC_Inverter:5281, F.Cu at (464.2, 55.6)
- added TP9: 5281, SiC_Inverter:5281, F.Cu at (368.8, 150.4)
- C58: value 10 uF -> 0.1 uF
- C59: value 18 pF -> 10 uF; footprint Capacitor_SMD:C_0402_1005Metric_Pad0.74x0.62mm_HandSolder -> Capacitor_SMD:C_0805_2012Metric_Pad1.18x1.45mm_HandSolder
- C60: value 18 pF -> 0.1 uF; footprint Capacitor_SMD:C_0402_1005Metric_Pad0.74x0.62mm_HandSolder -> Capacitor_SMD:C_0805_2012Metric_Pad1.18x1.45mm_HandSolder
- C64, C65: value 0.1 uF -> 18 pF; footprint Capacitor_SMD:C_0805_2012Metric_Pad1.18x1.45mm_HandSolder -> Capacitor_SMD:C_0402_1005Metric_Pad0.74x0.62mm_HandSolder
- C66: value 1 uF -> 0.1 uF; footprint Capacitor_SMD:C_1206_3216Metric_Pad1.33x1.80mm_HandSolder -> Capacitor_SMD:C_0805_2012Metric_Pad1.18x1.45mm_HandSolder
- C67: value 0.1 uF -> 10 uF
- C68: value 10 uF -> 1 uF; footprint Capacitor_SMD:C_0805_2012Metric_Pad1.18x1.45mm_HandSolder -> Capacitor_SMD:C_1206_3216Metric_Pad1.33x1.80mm_HandSolder
- IC2: value TPD2EUSB30ADRTR -> CP2102N-A02-GQFN24R; footprint SiC_Inverter:TPD2EUSB30ADRTR -> SiC_Inverter:CP2102N-A02-GQFN24R
- IC3: value CP2102N-A02-GQFN24R -> TPD2EUSB30ADRTR; footprint SiC_Inverter:CP2102N-A02-GQFN24R -> SiC_Inverter:TPD2EUSB30ADRTR
- J12, J20: value 43650-0418 -> 43045-1212; footprint SiC_Inverter:436500418 -> SiC_Inverter:43045-1212
- J13: value 464369202 -> 43650-0418; footprint SiC_Inverter:46436-900_02 -> SiC_Inverter:436500418
- J14: value 464379202 -> 43650-0418; footprint SiC_Inverter:46437-900_02 -> SiC_Inverter:436500418
- J15: value 43650-0418 -> 464369202; footprint SiC_Inverter:436500418 -> SiC_Inverter:46436-900_02
- J16: value 464369202 -> 464379202; footprint SiC_Inverter:46436-900_02 -> SiC_Inverter:46437-900_02
- J22: value 43045-1212 -> 464369202; footprint SiC_Inverter:43045-1212 -> SiC_Inverter:46436-900_02
- J23: value 43045-1212 -> 43650-0418; footprint SiC_Inverter:43045-1212 -> SiC_Inverter:436500418
- J24: value 1051330011 -> 43650-0418; footprint SiC_Inverter:105133-0011 -> SiC_Inverter:436500418
- R33: value 47 -> 100K
- R40: value 100K -> 47
- R42: value 0 -> 100K
- R43: value 100K -> 0
- moved PS1 171.2 mm to (470.4, 81.8)
- moved PS2 171.2 mm to (470.4, 107.3)
- moved J16 166.7 mm to (347.3, 54.0)
- moved J8 163.1 mm to (483.5, 30.9)
- moved U5 161.9 mm to (493.8, 111.9)
- moved J24 161.7 mm to (503.9, 83.1)
- moved C37 157.2 mm to (334.2, 169.6)
- moved C38 157.2 mm to (334.2, 172.6)
- moved C41 157.2 mm to (335.7, 192.5)
- moved C42 157.2 mm to (335.7, 195.0)
- moved C43 157.2 mm to (335.7, 197.5)
- moved C44 157.2 mm to (334.2, 175.6)
- moved C46 157.2 mm to (335.7, 200.0)
- moved C47 157.2 mm to (334.2, 178.6)
- moved C48 157.2 mm to (334.2, 181.6)
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Connections:
- C59 pad 1: Net-(Y1-GND_1) -> +3V3
- C60 pad 1: Net-(Y1-GND_2) -> +3V3
- C64 pad 1: +3V3 -> Net-(Y1-GND_1)
- C65 pad 1: +3V3 -> Net-(Y1-GND_2)
- C66 pad 1: /USB_Console/USB_VBUS -> +3V3
- C68 pad 1: +3V3 -> /USB_Console/USB_VBUS
- IC2 pad 1: /USB_Console/USBESP_D+ -> unconnected-(IC2-RI_/_CLK-Pad1)
- IC2 pad 2: /USB_Console/USBESP_D- -> LOGIC_GND
- IC2 pad 3: LOGIC_GND -> /USB_Console/USBESP_D+
- IC3 pad 1: unconnected-(IC3-RI_/_CLK-Pad1) -> /USB_Console/USBESP_D+
- IC3 pad 2: LOGIC_GND -> /USB_Console/USBESP_D-
- IC3 pad 3: /USB_Console/USBESP_D+ -> LOGIC_GND
- J12 pad 1: GND_ISO_LBHS -> /Con_RDY_A_L
- J12 pad 2: +15V_ISO_LBLS -> /Con_RDY_A_H
- J12 pad 3: GND_ISO_LAHS -> /Con_FLT_A_L
- J12 pad 4: +15V_ISO_LALS -> /Con_FLT_A_H
- J16 pad P1_1: /EMI_Input_Filter/+VIN_EMI -> GND_ISO_LBHS
- J16 pad P1_10: /EMI_Input_Filter/+VIN_EMI -> GND_ISO_LBHS
- J16 pad P1_2: /EMI_Input_Filter/+VIN_EMI -> GND_ISO_LBHS
- J16 pad P1_3: /EMI_Input_Filter/+VIN_EMI -> GND_ISO_LBHS
- J16 pad P1_4: /EMI_Input_Filter/+VIN_EMI -> GND_ISO_LBHS
- J16 pad P1_5: /EMI_Input_Filter/+VIN_EMI -> GND_ISO_LBHS
- J16 pad P1_6: /EMI_Input_Filter/+VIN_EMI -> GND_ISO_LBHS
- J16 pad P1_7: /EMI_Input_Filter/+VIN_EMI -> GND_ISO_LBHS
- J16 pad P1_8: /EMI_Input_Filter/+VIN_EMI -> GND_ISO_LBHS
- J16 pad P1_9: /EMI_Input_Filter/+VIN_EMI -> GND_ISO_LBHS
- J16 pad P2_1: GND -> GND_ISO_LAHS
- J16 pad P2_10: GND -> GND_ISO_LAHS
- J16 pad P2_2: GND -> GND_ISO_LAHS
- J16 pad P2_3: GND -> GND_ISO_LAHS
- J16 pad P2_4: GND -> GND_ISO_LAHS
- J16 pad P2_5: GND -> GND_ISO_LAHS
- J16 pad P2_6: GND -> GND_ISO_LAHS
- J16 pad P2_7: GND -> GND_ISO_LAHS
- J16 pad P2_8: GND -> GND_ISO_LAHS
- J16 pad P2_9: GND -> GND_ISO_LAHS
- J18 pad 1: GND_ISO_LBHS -> /Con_PWM_A_H
- J18 pad 2: +15V_ISO_LBLS -> /Con_PWM_A_L
- J18 pad 3: GND_ISO_LAHS -> /Con_PWM_B_H
- J18 pad 4: +15V_ISO_LBLS -> /Con_PWM_B_L
- J20 pad 1: /Con_PWM_A_H -> /Con_RDY_A_L
- J20 pad 2: /Con_PWM_A_L -> /Con_RDY_A_H
- J20 pad 3: /Con_PWM_B_H -> /Con_FLT_A_L
- J20 pad 4: /Con_PWM_B_L -> /Con_FLT_A_H
- J21 pad 1: /Full-Bridge/ePWM_A_H -> GND
- J21 pad 2: /Full-Bridge/ePWM_A_L -> /EMI_Input_Filter/+VIN_EMI
- J21 pad 3: /Full-Bridge/ePWM_B_H -> /EMI_Input_Filter/+VIN_EMI
- J21 pad 4: /Full-Bridge/ePWM_B_L -> unconnected-(J21-Pad4)
- J23 pad 1: /Con_RDY_A_L -> GND
- J23 pad 2: /Con_RDY_A_H -> /EMI_Input_Filter/+VIN_EMI
- J23 pad 3: /Con_FLT_A_L -> /EMI_Input_Filter/+VIN_EMI
- J23 pad 4: /Con_FLT_A_H -> unconnected-(J23-Pad4)
- J24 pad 1: /USB_Console/USB_VBUS -> LOGIC_GND
- J24 pad 2: /USB_Console/USB_D- -> +3V3
- J24 pad 3: /USB_Console/USB_D+ -> unconnected-(J24-Pad3)
- PS1 pad 1: /Power/DC+_IN_1 -> /EMI_Input_Filter/+VIN_EMI
- PS2 pad 1: /Power/DC+_IN_2 -> /EMI_Input_Filter/+VIN_EMI
- R33 pad 1: Net-(Q6-G) -> +3V3
- R33 pad 2: GND -> /Con_SCIRXDA
- R34 pad 1: GND -> +3V3
- R34 pad 2: GND -> /Controller/Flash_Boot_PU
- R35 pad 2: /Controller/Flash_Boot_PU -> /Controller/XRSn
- R37 pad 1: +3V3 -> /Controller/Flash_Boot_PD
- R37 pad 2: /Controller/TDI -> LOGIC_GND
- R38 pad 1: /Controller/TCK -> +3V3
- R38 pad 2: LOGIC_GND -> /Controller/TDI
- R39 pad 1: +3V3 -> /Controller/TCK
- R39 pad 2: /Controller/XRSn -> LOGIC_GND
- R40 pad 1: /Controller/Flash_Boot_PD -> Net-(Q6-G)
- R40 pad 2: LOGIC_GND -> GND
- R41 pad 1: +3V3 -> GND
- R41 pad 2: /Con_SCIRXDA -> GND
- R42 pad 1: LOGIC_GND -> +3V3
- R42 pad 2: Net-(J24-GND) -> Net-(IC2-RSTB)
- R43 pad 1: +3V3 -> LOGIC_GND
- R43 pad 2: Net-(IC3-RSTB) -> Net-(J26-GND)
Other:
- board size 204.5 x 65.2 mm -> 226.1 x 209.5 mm

Commit message: [WIP Input Protection Circuit to Controller]
- Added Gate node input protection pin to controller
- Added optocoupler to input protection circuit
- Added 3d model for PC817.....
- Updated PCB to test out PCB modularity
Parts:
- added C69: 0.1 uF, Capacitor_SMD:C_0805_2012Metric_Pad1.18x1.45mm_HandSolder, F.Cu at (59.0, 37.5)
- added Q7: PC817X1CSP9F, SiC_Inverter:PC817X1CSP9F, F.Cu at (492.7, 124.9)
- added R44: 499 K, Resistor_SMD:R_1206_3216Metric_Pad1.30x1.75mm_HandSolder, F.Cu at (46.5, 38.5)
- added R45: 499 K, Resistor_SMD:R_1206_3216Metric_Pad1.30x1.75mm_HandSolder, F.Cu at (52.0, 38.5)
- added R46: 10 K, Resistor_SMD:R_1206_3216Metric_Pad1.30x1.75mm_HandSolder, F.Cu at (457.4, 146.4)
- added R47: 10 K, Resistor_SMD:R_1206_3216Metric_Pad1.30x1.75mm_HandSolder, F.Cu at (457.4, 149.7)
- added TP54: 5277, SiC_Inverter:5277, F.Cu at (65.5, 59.5)
- added TP55: 5277, SiC_Inverter:5277, F.Cu at (507.2, 29.6)
- R18, R19, R3, R33, R34, R35, R36, R37, R38, R39, R4, R41, R42, R5: value 100K -> 100 K
- moved F1 468.5 mm to (38.5, 47.0)
- moved D6 457.5 mm to (54.5, 43.0)
- moved D5 456.1 mm to (42.6, 33.5)
- moved Q6 443.8 mm to (54.0, 55.9), turned to -90 degrees
- moved R41 422.9 mm to (61.5, 37.0), turned to -90 degrees
- moved R40 421.7 mm to (59.0, 42.5), turned to 90 degrees
- moved TP46 417.7 mm to (76.5, 27.0), turned to 90 degrees
- moved TP47 408.9 mm to (76.5, 59.5), turned to 90 degrees
- moved J22 400.2 mm to (76.0, 46.5), turned to 90 degrees
- moved J2 389.7 mm to (32.5, 57.5), turned to 90 degrees
- moved J1 384.8 mm to (32.4, 29.6), turned to 90 degrees
- moved TP1 374.9 mm to (43.5, 27.5), turned to 90 degrees
- moved TP2 366.3 mm to (43.5, 59.5), turned to 90 degrees
- moved J5 351.3 mm to (95.5, 38.0), turned to -90 degrees
- moved C1 315.7 mm to (112.2, 58.9), turned to 180 degrees
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Connections:
- D6 pad 1: GND -> /Con_Pro_Gate_node_output
- IC1 pad 32: unconnected-(IC1-GPIO33-Pad32) -> /Controller/Con_Gate_node_input
- J17 pad 4: unconnected-(J17-Pad4) -> /Con_Pro_Gate_node_output
- J21 pad 4: unconnected-(J21-Pad4) -> /Con_Pro_Gate_node_output
- J23 pad 4: unconnected-(J23-Pad4) -> /Con_Pro_Gate_node_output
- J24 pad 4: unconnected-(J24-Pad4) -> /Con_Pro_Gate_node_output
- R40 pad 2: GND -> /Con_Pro_Gate_node_output
- R41 pad 2: GND -> /Con_Pro_Gate_node_output

Commit message: Added Precharge Gate Driver to controller and per charge sub circuit
Parts:
- added D7: BZX84C15-7-F, Package_TO_SOT_SMD:SOT-23-3, F.Cu at (525.2, 25.0)
- added J27: 43650-0418, SiC_Inverter:436500418, F.Cu at (508.5, 158.5)
- added J28: 43650-0418, SiC_Inverter:436500418, F.Cu at (525.5, 16.5)
- added Q8: PC817X1CSP9F, SiC_Inverter:PC817X1CSP9F, F.Cu at (506.5, 150.0)
- added R48: 499 K, Resistor_SMD:R_1206_3216Metric_Pad1.30x1.75mm_HandSolder, F.Cu at (519.7, 24.4)
- added R49: 2 K, Resistor_SMD:R_1206_3216Metric_Pad1.30x1.75mm_HandSolder, F.Cu at (510.5, 144.0)
Connections:
- IC1 pad 54: unconnected-(IC1-GPIO23_VSW-Pad54) -> /Controller/Con_Gate_node_prech
- J17 pad 3: unconnected-(J17-Pad3) -> GND
- J21 pad 4: /Con_Pro_Gate_node_output -> /Input_Protection/Gate_node_input_pro
- J24 pad 3: unconnected-(J24-Pad3) -> GND
- Q1 pad 1: Net-(Q1-G) -> Net-(D7-K)
- R2 pad 1: Net-(Q1-G) -> Net-(D7-K)
- R2 pad 2: /Pre-Chrage_current_Limiting/Gate_node_prech -> /Con_Gate_node_prech
- R3 pad 1: /DC_Link_Caps/BUS_DC+ -> /Con_Gate_node_prech
- R3 pad 2: Net-(Q1-G) -> GND
- TP55 pad 1: /Pre-Chrage_current_Limiting/Gate_node_prech -> /Con_Gate_node_prech
Other:
- board size 226.1 x 209.5 mm -> 285.6 x 209.5 mm

Commit message: WIP PCB, Added Test Points, added icon file
Parts:
- added G***: LOGO, SiC_Inverter:Inverter_PCB_Icon, B.Cu at (68.3, 101.7)
- added TP56: 5277, SiC_Inverter:5277, F.Cu at (449.1, 220.7)
- added TP57: 5277, SiC_Inverter:5277, F.Cu at (449.1, 227.0)
- added TP58: 5277, SiC_Inverter:5277, F.Cu at (449.1, 233.2)
- added TP59: 5281, SiC_Inverter:5281, F.Cu at (449.1, 239.5)
- added TP60: 5277, SiC_Inverter:5277, F.Cu at (449.1, 245.8)
- added TP61: 5277, SiC_Inverter:5277, F.Cu at (449.1, 252.0)
- added TP62: 5277, SiC_Inverter:5277, F.Cu at (455.3, 220.7)
- added TP63: 5277, SiC_Inverter:5277, F.Cu at (455.3, 227.0)
- added TP64: 5277, SiC_Inverter:5277, F.Cu at (455.3, 233.2)
- added TP65: 5277, SiC_Inverter:5277, F.Cu at (455.3, 239.5)
- added TP66: 5281, SiC_Inverter:5281, F.Cu at (455.3, 245.8)
- added TP67: 5277, SiC_Inverter:5277, F.Cu at (65.0, 60.5)
- added TP68: 5281, SiC_Inverter:5281, F.Cu at (82.0, 60.5)
- added TP69: 5277, SiC_Inverter:5277, F.Cu at (82.0, 28.0)
- added TP70: 5281, SiC_Inverter:5281, F.Cu at (578.4, 272.8)
- added TP71: 5277, SiC_Inverter:5277, F.Cu at (578.4, 279.1)
- added TP72: 5277, SiC_Inverter:5277, F.Cu at (584.6, 272.8)
- added TP73: 5281, SiC_Inverter:5281, F.Cu at (584.6, 279.1)
- added TP74: 5277, SiC_Inverter:5277, F.Cu at (590.9, 272.8)
- added TP75: 5281, SiC_Inverter:5281, F.Cu at (590.9, 279.1)
- C67: value 10 uF -> 0.1 uF
- C68: value 1 uF -> 10 uF; footprint Capacitor_SMD:C_1206_3216Metric_Pad1.33x1.80mm_HandSolder -> Capacitor_SMD:C_0805_2012Metric_Pad1.18x1.45mm_HandSolder
- C69: value 0.1 uF -> 1 uF; footprint Capacitor_SMD:C_0805_2012Metric_Pad1.18x1.45mm_HandSolder -> Capacitor_SMD:C_1206_3216Metric_Pad1.33x1.80mm_HandSolder
- D1: value BZX84C20-7-F -> BZX84C15-7-F
- D5: value P6KE500A-HF -> BZX84C20-7-F; footprint Diode_THT:D_DO-15_P12.70mm_Horizontal -> Package_TO_SOT_SMD:SOT-23-3
- D6: value BZX84C15-7-F -> P6KE500A-HF; footprint Package_TO_SOT_SMD:SOT-23-3 -> Diode_THT:D_DO-15_P12.70mm_Horizontal
- J10, J8: value 464369202 -> 464379202; footprint SiC_Inverter:46436-900_02 -> SiC_Inverter:46437-900_02
- J11, J16, J9: value 464379202 -> 464369202; footprint SiC_Inverter:46437-900_02 -> SiC_Inverter:46436-900_02
- J12: value 43045-1212 -> 464379202; footprint SiC_Inverter:43045-1212 -> SiC_Inverter:46437-900_02
- J13: value 43650-0418 -> 43045-1212; footprint SiC_Inverter:436500418 -> SiC_Inverter:43045-1212
- J15, J22: value 464369202 -> 43650-0418; footprint SiC_Inverter:46436-900_02 -> SiC_Inverter:436500418
- J17: value 43650-0418 -> 464379202; footprint SiC_Inverter:436500418 -> SiC_Inverter:46437-900_02
- J23: value 43650-0418 -> 464369202; footprint SiC_Inverter:436500418 -> SiC_Inverter:46436-900_02
- J26: value 1051330011 -> 43650-0418; footprint SiC_Inverter:105133-0011 -> SiC_Inverter:436500418
- J28: value 43650-0418 -> 1051330011; footprint SiC_Inverter:436500418 -> SiC_Inverter:105133-0011
- J7: value 464379202 -> 43650-0418; footprint SiC_Inverter:46437-900_02 -> SiC_Inverter:436500418
- Q6: value STB10NK60ZT4 -> PC817X1CSP9F; footprint Package_TO_SOT_SMD:TO-263-2 -> SiC_Inverter:PC817X1CSP9F
- Q8: value PC817X1CSP9F -> STB10NK60ZT4; footprint SiC_Inverter:PC817X1CSP9F -> Package_TO_SOT_SMD:TO-263-2
- R1: value CW005100R0JE12HE -> 499 K; footprint SiC_Inverter:CW005100R0JE12HE -> Resistor_SMD:R_1206_3216Metric_Pad1.30x1.75mm_HandSolder
- R10, R24: value 5 K -> 10
- R11, R14, R25, R28: value 100 -> 5 K
- R12, R15, R26, R29: value 5 K -> 100
- R18: value 100 K -> 5 K
- R2: value 47 -> CW005100R0JE12HE; footprint Resistor_SMD:R_1206_3216Metric_Pad1.30x1.75mm_HandSolder -> SiC_Inverter:CW005100R0JE12HE
- R20, R6: value 10 -> 100 K
- R3: value 100 K -> 47
- R32: value R -> 5 K; footprint SiC_Inverter:CW005100R0JE12HE -> Resistor_SMD:R_1206_3216Metric_Pad1.30x1.75mm_HandSolder
- R33: value 100 K -> R; footprint Resistor_SMD:R_1206_3216Metric_Pad1.30x1.75mm_HandSolder -> SiC_Inverter:CW005100R0JE12HE
- R35, R42: value 100 K -> 10 K
- R38: value 100 K -> 2 K
- R40: value 47 -> 100 K
- R43: value 0 -> 100 K
- R46: value 10 K -> 47
- R47: value 10 K -> 100 K
- R48: value 499 K -> 100 K
- R49: value 2 K -> 0
- TP10, TP31, TP33, TP39: value 5277 -> 5281; footprint SiC_Inverter:5277 -> SiC_Inverter:5281
- TP29, TP32, TP43, TP45, TP47, TP48, TP50, TP52, TP8: value 5281 -> 5277; footprint SiC_Inverter:5281 -> SiC_Inverter:5277
- moved J5 531.7 mm to (597.0, 214.5), turned to 0 degrees
- moved C69 483.9 mm to (492.6, 252.2), turned to 0 degrees
- moved C1 482.1 mm to (575.8, 190.9), turned to 0 degrees
- moved L1 469.2 mm to (543.5, 219.9)
- moved TP5 468.7 mm to (598.0, 182.0)
- moved D7 464.4 mm to (61.0, 38.0), turned to 90 degrees
- moved Q8 464.1 mm to (52.0, 56.1), turned to -90 degrees
- moved Q6 461.6 mm to (464.9, 266.3), turned to 0 degrees
- moved C66 460.1 mm to (64.5, 38.5), turned to -90 degrees
- moved TP6 457.4 mm to (598.0, 188.2)
- moved J6 452.8 mm to (580.0, 214.5), turned to 0 degrees
- moved R41 449.6 mm to (461.4, 242.4), turned to 0 degrees
- moved J24 447.9 mm to (67.3, 28.3)
- moved R40 447.9 mm to (461.4, 239.1), turned to 0 degrees
- moved J22 447.0 mm to (478.6, 240.8), turned to 0 degrees
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Connections:
- C66 pad 1: +3V3 -> GND
- C66 pad 2: LOGIC_GND -> /Con_Pro_Gate_node_output
- C68 pad 1: /USB_Console/USB_VBUS -> +3V3
- C69 pad 1: GND -> /USB_Console/USB_VBUS
- C69 pad 2: /Con_Pro_Gate_node_output -> LOGIC_GND
- D1 pad 1: /Full-Bridge/Leg_A_Power_Stage/LegA_HS_Gate -> Net-(D1-K)
- D1 pad 2: GND_ISO_LAHS -> /DC_Link_Caps/BUS_DC+
- D2 pad 1: /Full-Bridge/Leg_A_Power_Stage/LegA_LS_Gate -> /Full-Bridge/Leg_A_Power_Stage/LegA_HS_Gate
- D3 pad 1: /Full-Bridge/Leg_B_Power_Stage/LegB_HS_Gate -> /Full-Bridge/Leg_A_Power_Stage/LegA_LS_Gate
- D3 pad 2: GND_ISO_LBHS -> GND_ISO_LAHS
- D4 pad 1: /Full-Bridge/Leg_B_Power_Stage/LegB_LS_Gate -> /Full-Bridge/Leg_B_Power_Stage/LegB_HS_Gate
- D5 pad 1: /EMI_Input_Filter/+VIN_EMI -> /Full-Bridge/Leg_B_Power_Stage/LegB_LS_Gate
- D5 pad 2: GND -> GND_ISO_LBHS
- D6 pad 1: /Con_Pro_Gate_node_output -> /EMI_Input_Filter/+VIN_EMI
- D7 pad 1: Net-(D7-K) -> /Con_Pro_Gate_node_output
- D7 pad 2: /DC_Link_Caps/BUS_DC+ -> GND
- J10 pad P1_1: /DC_Link_Caps/BUS_DC+ -> GND
- J10 pad P1_10: /DC_Link_Caps/BUS_DC+ -> GND
- J10 pad P1_2: /DC_Link_Caps/BUS_DC+ -> GND
- J10 pad P1_3: /DC_Link_Caps/BUS_DC+ -> GND
- J10 pad P1_4: /DC_Link_Caps/BUS_DC+ -> GND
- J10 pad P1_5: /DC_Link_Caps/BUS_DC+ -> GND
- J10 pad P1_6: /DC_Link_Caps/BUS_DC+ -> GND
- J10 pad P1_7: /DC_Link_Caps/BUS_DC+ -> GND
- J10 pad P1_8: /DC_Link_Caps/BUS_DC+ -> GND
- J10 pad P1_9: /DC_Link_Caps/BUS_DC+ -> GND
- J10 pad P2_1: GND -> /DC_Link_Caps/BUS_DC+
- J10 pad P2_10: GND -> /DC_Link_Caps/BUS_DC+
- J10 pad P2_2: GND -> /DC_Link_Caps/BUS_DC+
- J10 pad P2_3: GND -> /DC_Link_Caps/BUS_DC+
- J10 pad P2_4: GND -> /DC_Link_Caps/BUS_DC+
- J10 pad P2_5: GND -> /DC_Link_Caps/BUS_DC+
- J10 pad P2_6: GND -> /DC_Link_Caps/BUS_DC+
- J10 pad P2_7: GND -> /DC_Link_Caps/BUS_DC+
- J10 pad P2_8: GND -> /DC_Link_Caps/BUS_DC+
- J10 pad P2_9: GND -> /DC_Link_Caps/BUS_DC+
- J11 pad P1_1: GND -> /DC_Link_Caps/BUS_DC+
- J11 pad P1_10: GND -> /DC_Link_Caps/BUS_DC+
- J11 pad P1_2: GND -> /DC_Link_Caps/BUS_DC+
- J11 pad P1_3: GND -> /DC_Link_Caps/BUS_DC+
- J11 pad P1_4: GND -> /DC_Link_Caps/BUS_DC+
- J11 pad P1_5: GND -> /DC_Link_Caps/BUS_DC+
- J11 pad P1_6: GND -> /DC_Link_Caps/BUS_DC+
- J11 pad P1_7: GND -> /DC_Link_Caps/BUS_DC+
- J11 pad P1_8: GND -> /DC_Link_Caps/BUS_DC+
- J11 pad P1_9: GND -> /DC_Link_Caps/BUS_DC+
- J11 pad P2_1: /DC_Link_Caps/BUS_DC+ -> GND
- J11 pad P2_10: /DC_Link_Caps/BUS_DC+ -> GND
- J11 pad P2_2: /DC_Link_Caps/BUS_DC+ -> GND
- J11 pad P2_3: /DC_Link_Caps/BUS_DC+ -> GND
- J11 pad P2_4: /DC_Link_Caps/BUS_DC+ -> GND
- J11 pad P2_5: /DC_Link_Caps/BUS_DC+ -> GND
- J11 pad P2_6: /DC_Link_Caps/BUS_DC+ -> GND
- J11 pad P2_7: /DC_Link_Caps/BUS_DC+ -> GND
- J11 pad P2_8: /DC_Link_Caps/BUS_DC+ -> GND
- J11 pad P2_9: /DC_Link_Caps/BUS_DC+ -> GND
- J13 pad 1: /Con_PWM_A_H -> /Con_RDY_A_L
- J13 pad 2: /Con_PWM_A_L -> /Con_RDY_A_H
- J13 pad 3: /Con_PWM_B_H -> /Con_FLT_A_L
- J13 pad 4: /Con_PWM_B_L -> /Con_FLT_A_H
- J14 pad 1: GND_ISO_LBHS -> /Con_PWM_A_H
- J14 pad 2: +15V_ISO_LBLS -> /Con_PWM_A_L
- J14 pad 3: GND_ISO_LAHS -> /Con_PWM_B_H
- J14 pad 4: +15V_ISO_LALS -> /Con_PWM_B_L
- J16 pad P1_1: GND_ISO_LBHS -> GND_ISO_LAHS
- J16 pad P1_10: GND_ISO_LBHS -> GND_ISO_LAHS
- J16 pad P1_2: GND_ISO_LBHS -> GND_ISO_LAHS
- J16 pad P1_3: GND_ISO_LBHS -> GND_ISO_LAHS
- J16 pad P1_4: GND_ISO_LBHS -> GND_ISO_LAHS
- J16 pad P1_5: GND_ISO_LBHS -> GND_ISO_LAHS
- J16 pad P1_6: GND_ISO_LBHS -> GND_ISO_LAHS
- J16 pad P1_7: GND_ISO_LBHS -> GND_ISO_LAHS
- J16 pad P1_8: GND_ISO_LBHS -> GND_ISO_LAHS
- J16 pad P1_9: GND_ISO_LBHS -> GND_ISO_LAHS
- J16 pad P2_1: GND_ISO_LAHS -> GND_ISO_LBHS
- J16 pad P2_10: GND_ISO_LAHS -> GND_ISO_LBHS
- J16 pad P2_2: GND_ISO_LAHS -> GND_ISO_LBHS
- J16 pad P2_3: GND_ISO_LAHS -> GND_ISO_LBHS
- J16 pad P2_4: GND_ISO_LAHS -> GND_ISO_LBHS
- J16 pad P2_5: GND_ISO_LAHS -> GND_ISO_LBHS
- J16 pad P2_6: GND_ISO_LAHS -> GND_ISO_LBHS
- J16 pad P2_7: GND_ISO_LAHS -> GND_ISO_LBHS
- J16 pad P2_8: GND_ISO_LAHS -> GND_ISO_LBHS
- J16 pad P2_9: GND_ISO_LAHS -> GND_ISO_LBHS
- J18 pad 1: /Con_PWM_A_H -> LOGIC_GND
- J18 pad 2: /Con_PWM_A_L -> +3V3
- J18 pad 3: /Con_PWM_B_H -> GND
- J18 pad 4: /Con_PWM_B_L -> /Con_Pro_Gate_node_output
- J21 pad 1: GND -> /Con_PWM_A_H
- J21 pad 2: /EMI_Input_Filter/+VIN_EMI -> /Con_PWM_A_L
- J21 pad 3: /EMI_Input_Filter/+VIN_EMI -> /Con_PWM_B_H
- J21 pad 4: /Input_Protection/Gate_node_input_pro -> /Con_PWM_B_L
- J24 pad 1: LOGIC_GND -> GND
- J24 pad 2: +3V3 -> /EMI_Input_Filter/+VIN_EMI
- J24 pad 3: GND -> /EMI_Input_Filter/+VIN_EMI
- J25 pad 1: GND_ISO_LBHS -> GND
- J25 pad 2: +15V_ISO_LBLS -> /EMI_Input_Filter/+VIN_EMI
- J25 pad 3: GND_ISO_LAHS -> /EMI_Input_Filter/+VIN_EMI
- J25 pad 4: +15V_ISO_LBLS -> /Con_Pro_Gate_node_output
- J26 pad 1: /USB_Console/USB_VBUS -> LOGIC_GND
- J26 pad 2: /USB_Console/USB_D- -> +3V3
- J26 pad 3: /USB_Console/USB_D+ -> GND
- J26 pad 4: unconnected-(J26-ID-Pad4) -> /Con_Pro_Gate_node_output
- J27 pad 1: /Con_Gate_node_prech -> GND_ISO_LBHS
- J27 pad 2: GND -> +15V_ISO_LBLS
- J27 pad 3: unconnected-(J27-Pad3) -> GND_ISO_LAHS
- J27 pad 4: unconnected-(J27-Pad4) -> +15V_ISO_LBLS
- J28 pad 1: /Con_Gate_node_prech -> /USB_Console/USB_VBUS
- J28 pad 2: GND -> /USB_Console/USB_D-
- J28 pad 3: unconnected-(J28-Pad3) -> /USB_Console/USB_D+
- J8 pad P1_1: /DC_Link_Caps/BUS_DC+ -> GND
- J8 pad P1_10: /DC_Link_Caps/BUS_DC+ -> GND
- J8 pad P1_2: /DC_Link_Caps/BUS_DC+ -> GND
- J8 pad P1_3: /DC_Link_Caps/BUS_DC+ -> GND
- J8 pad P1_4: /DC_Link_Caps/BUS_DC+ -> GND
- J8 pad P1_5: /DC_Link_Caps/BUS_DC+ -> GND
- J8 pad P1_6: /DC_Link_Caps/BUS_DC+ -> GND
- J8 pad P1_7: /DC_Link_Caps/BUS_DC+ -> GND
- J8 pad P1_8: /DC_Link_Caps/BUS_DC+ -> GND
- J8 pad P1_9: /DC_Link_Caps/BUS_DC+ -> GND
- J8 pad P2_1: GND -> /EMI_Input_Filter/BUS+_Filtered
- J8 pad P2_10: GND -> /EMI_Input_Filter/BUS+_Filtered
- J8 pad P2_2: GND -> /EMI_Input_Filter/BUS+_Filtered
- J8 pad P2_3: GND -> /EMI_Input_Filter/BUS+_Filtered
- J8 pad P2_4: GND -> /EMI_Input_Filter/BUS+_Filtered
- J8 pad P2_5: GND -> /EMI_Input_Filter/BUS+_Filtered
- J8 pad P2_6: GND -> /EMI_Input_Filter/BUS+_Filtered
- J8 pad P2_7: GND -> /EMI_Input_Filter/BUS+_Filtered
- J8 pad P2_8: GND -> /EMI_Input_Filter/BUS+_Filtered
- J8 pad P2_9: GND -> /EMI_Input_Filter/BUS+_Filtered
- J9 pad P1_1: GND -> /DC_Link_Caps/BUS_DC+
- J9 pad P1_10: GND -> /DC_Link_Caps/BUS_DC+
- J9 pad P1_2: GND -> /DC_Link_Caps/BUS_DC+
- J9 pad P1_3: GND -> /DC_Link_Caps/BUS_DC+
- J9 pad P1_4: GND -> /DC_Link_Caps/BUS_DC+
- J9 pad P1_5: GND -> /DC_Link_Caps/BUS_DC+
- J9 pad P1_6: GND -> /DC_Link_Caps/BUS_DC+
- J9 pad P1_7: GND -> /DC_Link_Caps/BUS_DC+
- J9 pad P1_8: GND -> /DC_Link_Caps/BUS_DC+
- J9 pad P1_9: GND -> /DC_Link_Caps/BUS_DC+
- J9 pad P2_1: /DC_Link_Caps/BUS_DC+ -> GND
- J9 pad P2_10: /DC_Link_Caps/BUS_DC+ -> GND
- J9 pad P2_2: /DC_Link_Caps/BUS_DC+ -> GND
- J9 pad P2_3: /DC_Link_Caps/BUS_DC+ -> GND
- J9 pad P2_4: /DC_Link_Caps/BUS_DC+ -> GND
- J9 pad P2_5: /DC_Link_Caps/BUS_DC+ -> GND
- J9 pad P2_6: /DC_Link_Caps/BUS_DC+ -> GND
- J9 pad P2_7: /DC_Link_Caps/BUS_DC+ -> GND
- J9 pad P2_8: /DC_Link_Caps/BUS_DC+ -> GND
- J9 pad P2_9: /DC_Link_Caps/BUS_DC+ -> GND
- Q1 pad 1: Net-(D7-K) -> Net-(D1-K)
- Q6 pad 1: Net-(Q6-G) -> Net-(Q6-A)
- Q6 pad 2: -VIN -> GND
- Q6 pad 3: GND -> /Controller/Con_Gate_node_input
- Q7 pad 2: GND -> /Controller/Con_Gate_node_prech
- Q7 pad 3: /Controller/Con_Gate_node_input -> GND
- Q7 pad 4: LOGIC_GND -> /Con_Gate_node_prech
- Q8 pad 1: Net-(Q8-A) -> Net-(Q8-G)
- Q8 pad 2: /Controller/Con_Gate_node_prech -> -VIN
- R1 pad 2: /DC_Link_Caps/BUS_DC+ -> /Con_Gate_node_prech
- R10 pad 1: +3V3 -> /Full-Bridge/Leg_A_Power_Stage/LegA_LS_OUTL
- R10 pad 2: /Con_EN_A_L -> /Full-Bridge/Leg_A_Power_Stage/LegA_LS_Gate
- R11 pad 1: Net-(U1-IN+) -> +3V3
- R11 pad 2: /Con_PWM_A_L -> /Con_EN_A_L
- R12 pad 1: +3V3 -> Net-(U1-IN+)
- R12 pad 2: /Con_EN_A_H -> /Con_PWM_A_L
- R13 pad 2: /Con_FLT_A_L -> /Con_EN_A_H
- R14 pad 1: Net-(U2-IN+) -> +3V3
- R14 pad 2: /Con_PWM_A_H -> /Con_FLT_A_L
- R15 pad 1: +3V3 -> Net-(U2-IN+)
- R15 pad 2: /Con_FLT_A_H -> /Con_PWM_A_H
- R16 pad 2: /Con_RDY_A_L -> /Con_FLT_A_H
- R17 pad 2: /Con_RDY_A_H -> /Con_RDY_A_L
- R18 pad 1: /Full-Bridge/Leg_B_Power_Stage/LegB_HS_Gate -> +3V3
- R18 pad 2: GND_ISO_LBHS -> /Con_RDY_A_H
- R19 pad 1: /Full-Bridge/Leg_B_Power_Stage/LegB_LS_Gate -> /Full-Bridge/Leg_B_Power_Stage/LegB_HS_Gate
- R2 pad 1: Net-(D7-K) -> /EMI_Input_Filter/BUS+_Filtered
- R2 pad 2: /Con_Gate_node_prech -> /DC_Link_Caps/BUS_DC+
- R20 pad 1: /Full-Bridge/Leg_B_Power_Stage/LegB_HS_OUTH -> /Full-Bridge/Leg_B_Power_Stage/LegB_LS_Gate
- R20 pad 2: /Full-Bridge/Leg_B_Power_Stage/LegB_HS_Gate -> GND_ISO_LBHS
- R21 pad 1: /Full-Bridge/Leg_B_Power_Stage/LegB_HS_OUTL -> /Full-Bridge/Leg_B_Power_Stage/LegB_HS_OUTH
- R22 pad 1: /Full-Bridge/Leg_B_Power_Stage/LegB_LS_OUTH -> /Full-Bridge/Leg_B_Power_Stage/LegB_HS_OUTL
- R22 pad 2: /Full-Bridge/Leg_B_Power_Stage/LegB_LS_Gate -> /Full-Bridge/Leg_B_Power_Stage/LegB_HS_Gate
- R23 pad 1: /Full-Bridge/Leg_B_Power_Stage/LegB_LS_OUTL -> /Full-Bridge/Leg_B_Power_Stage/LegB_LS_OUTH
- R24 pad 1: +3V3 -> /Full-Bridge/Leg_B_Power_Stage/LegB_LS_OUTL
- R24 pad 2: /Con_EN_B_L -> /Full-Bridge/Leg_B_Power_Stage/LegB_LS_Gate
- R25 pad 1: Net-(U3-IN+) -> +3V3
- R25 pad 2: /Con_PWM_B_L -> /Con_EN_B_L
- R26 pad 1: +3V3 -> Net-(U3-IN+)
- R26 pad 2: /Con_EN_B_H -> /Con_PWM_B_L
- R27 pad 2: /Con_FLT_B_L -> /Con_EN_B_H
- R28 pad 1: Net-(U4-IN+) -> +3V3
- R28 pad 2: /Con_PWM_B_H -> /Con_FLT_B_L
- R29 pad 1: +3V3 -> Net-(U4-IN+)
- R29 pad 2: /Con_FLT_B_H -> /Con_PWM_B_H
- R3 pad 1: /Con_Gate_node_prech -> Net-(D1-K)
- R3 pad 2: GND -> /Con_Gate_node_prech
- R30 pad 2: /Con_RDY_B_L -> /Con_FLT_B_H
- R31 pad 2: /Con_RDY_B_H -> /Con_RDY_B_L
- R32 pad 1: /Phase_A_Output -> +3V3
- R32 pad 2: /Phase_B_Output -> /Con_RDY_B_H
- R33 pad 1: +3V3 -> /Phase_A_Output
- R33 pad 2: /Con_SCIRXDA -> /Phase_B_Output
- R34 pad 2: /Controller/Flash_Boot_PU -> /Con_SCIRXDA
- R35 pad 1: +3V3 -> /Con_Pro_Gate_node_output
- R35 pad 2: /Controller/XRSn -> Net-(Q6-A)
- R36 pad 2: /Controller/TMS -> /Controller/Flash_Boot_PU
- R37 pad 1: /Controller/Flash_Boot_PD -> +3V3
- R37 pad 2: LOGIC_GND -> /Controller/XRSn
- R38 pad 2: /Controller/TDI -> Net-(Q7-A)
- R39 pad 1: /Controller/TCK -> +3V3
- R39 pad 2: LOGIC_GND -> /Controller/TMS
- R4 pad 1: /Full-Bridge/Leg_A_Power_Stage/LegA_HS_Gate -> /Con_Gate_node_prech
- R4 pad 2: GND_ISO_LAHS -> GND
- R40 pad 1: Net-(Q6-G) -> /Controller/Flash_Boot_PD
- R40 pad 2: /Con_Pro_Gate_node_output -> LOGIC_GND
- R41 pad 1: GND -> +3V3
- R41 pad 2: /Con_Pro_Gate_node_output -> /Controller/TDI
- R42 pad 2: Net-(IC2-RSTB) -> /Controller/Con_Gate_node_input
- R43 pad 1: LOGIC_GND -> /Controller/TCK
- R43 pad 2: Net-(J26-GND) -> LOGIC_GND
- R46 pad 1: /Con_Pro_Gate_node_output -> Net-(Q8-G)
- R46 pad 2: Net-(Q7-A) -> /Con_Pro_Gate_node_output
- R47 pad 1: +3V3 -> GND
- R47 pad 2: /Controller/Con_Gate_node_input -> /Con_Pro_Gate_node_output
- R48 pad 1: /EMI_Input_Filter/BUS+_Filtered -> +3V3
- R48 pad 2: /Con_Gate_node_prech -> Net-(IC2-RSTB)
- R49 pad 1: +3V3 -> LOGIC_GND
- R49 pad 2: Net-(Q8-A) -> Net-(J28-GND)
- R5 pad 1: /Full-Bridge/Leg_A_Power_Stage/LegA_LS_Gate -> /Full-Bridge/Leg_A_Power_Stage/LegA_HS_Gate
- R6 pad 1: /Full-Bridge/Leg_A_Power_Stage/LegA_HS_OUTH -> /Full-Bridge/Leg_A_Power_Stage/LegA_LS_Gate
- R6 pad 2: /Full-Bridge/Leg_A_Power_Stage/LegA_HS_Gate -> GND_ISO_LAHS
- R7 pad 1: /Full-Bridge/Leg_A_Power_Stage/LegA_HS_OUTL -> /Full-Bridge/Leg_A_Power_Stage/LegA_HS_OUTH
- R8 pad 1: /Full-Bridge/Leg_A_Power_Stage/LegA_LS_OUTH -> /Full-Bridge/Leg_A_Power_Stage/LegA_HS_OUTL
- R8 pad 2: /Full-Bridge/Leg_A_Power_Stage/LegA_LS_Gate -> /Full-Bridge/Leg_A_Power_Stage/LegA_HS_Gate
- R9 pad 1: /Full-Bridge/Leg_A_Power_Stage/LegA_LS_OUTL -> /Full-Bridge/Leg_A_Power_Stage/LegA_LS_OUTH
- TP10 pad 1: /DC_Link_Caps/BUS_DC+ -> GND
- TP11 pad 1: /Con_EN_A_H -> /DC_Link_Caps/BUS_DC+
- TP13 pad 1: /Con_RDY_A_H -> /Con_FLT_A_L
- TP14 pad 1: /Con_FLT_A_H -> /Con_RDY_A_L
- TP15 pad 1: /Con_RDY_A_L -> /Con_EN_A_H
- TP16 pad 1: /Con_FLT_A_L -> /Con_FLT_A_H
- TP17 pad 1: /Con_FLT_B_H -> /Con_RDY_A_H
- TP18 pad 1: /Con_RDY_B_L -> /Con_EN_B_L
- TP19 pad 1: /Con_EN_B_H -> /Con_FLT_B_L
- TP20 pad 1: /Con_FLT_B_L -> /Con_RDY_B_L
- TP21 pad 1: /Con_EN_B_L -> /Con_EN_B_H
- TP22 pad 1: /Con_RDY_B_H -> /Con_FLT_B_H
- TP23 pad 1: /Con_PWM_B_L -> /Con_RDY_B_H
- TP24 pad 1: /Con_PWM_B_H -> /Con_PWM_B_L
- TP25 pad 1: /Con_PWM_A_L -> /Con_PWM_B_H
- TP26 pad 1: /Con_PWM_A_H -> /Con_PWM_A_L
- TP27 pad 1: +15V_ISO_LALS -> /Con_PWM_A_H
- TP28 pad 1: +15V_ISO_LBLS -> +15V_ISO_LALS
- TP29 pad 1: GND_ISO_LAHS -> +15V_ISO_LBLS
- TP30 pad 1: GND_ISO_LBHS -> GND_ISO_LAHS
- TP31 pad 1: GND_ISO_LAHS -> GND_ISO_LBHS
- TP32 pad 1: GND_ISO_LBHS -> GND_ISO_LAHS
- TP33 pad 1: /Full-Bridge/Leg_A_Power_Stage/LegA_HS_Gate -> GND_ISO_LBHS
- TP34 pad 1: /Full-Bridge/Leg_A_Power_Stage/LegA_LS_Gate -> /Full-Bridge/Leg_A_Power_Stage/LegA_HS_Gate
- TP35 pad 1: /Full-Bridge/Leg_B_Power_Stage/LegB_HS_Gate -> /Full-Bridge/Leg_A_Power_Stage/LegA_LS_Gate
- TP36 pad 1: /Full-Bridge/Leg_B_Power_Stage/LegB_LS_Gate -> unconnected-(TP36-Pad1)
- TP37 pad 1: /Controller/TMS -> unconnected-(TP37-Pad1)
- TP38 pad 1: /Controller/TDI -> +3V3
- TP39 pad 1: /Controller/TCK -> LOGIC_GND
- TP40 pad 1: /Controller/XRSn -> /Con_Pro_Gate_node_output
- TP41 pad 1: /Controller/TDO -> /Con_PWM_B_L
- TP42 pad 1: +3V3 -> /Con_PWM_A_L
- TP43 pad 1: LOGIC_GND -> /Con_EN_A_H
- TP44 pad 1: Net-(Y1-GND_1) -> /Con_FLT_A_H
- TP45 pad 1: /Controller/X1 -> /Con_RDY_A_H
- TP46 pad 1: /EMI_Input_Filter/+VIN_EMI -> /Con_PWM_B_H
- TP47 pad 1: GND -> /Con_PWM_A_H
- TP48 pad 1: LOGIC_GND -> /Con_EN_A_L
- TP49 pad 1: +3V3 -> /Con_FLT_A_L
- TP50 pad 1: GND_ISO_LAHS -> /Con_RDY_A_L
- TP51 pad 1: +15V_ISO_LBLS -> /Controller/TMS
- TP52 pad 1: GND_ISO_LBHS -> /Controller/TDO
- TP53 pad 1: +15V_ISO_LBLS -> /Controller/XRSn
- TP54 pad 1: /Con_Pro_Gate_node_output -> /Controller/TCK
- TP55 pad 1: /Con_Gate_node_prech -> /Controller/TDI
- TP7 pad 1: /DC_Link_Caps/BUS_DC+ -> /Con_Gate_node_prech
- TP8 pad 1: GND -> /DC_Link_Caps/BUS_DC+
Other:
- board size 285.6 x 209.5 mm -> 322.1 x 269.5 mm
- board text added: "Controller + USB"
- board text added: "DC Input & Input Protection Circuit"
- board text added: "DC Link Caps"
- board text added: "Full-Bridge"
- board text added: "Power"
- board text added: "Pre-Charge_Current_Limiting"

Commit message: WIP PCB Design: Finished DC Input / Protection Circuit
Parts:
- added H1: MountingHole, MountingHole:MountingHole_2.2mm_M2, F.Cu at (84.0, 56.0)
- added H2: MountingHole, MountingHole:MountingHole_2.2mm_M2, F.Cu at (84.0, 38.5)
- added H3: MountingHole, MountingHole:MountingHole_2.2mm_M2, F.Cu at (57.0, 56.0)
- added H4: MountingHole, MountingHole:MountingHole_2.2mm_M2, F.Cu at (57.0, 38.5)
- J1, J3: value 23AH8786-Red -> CONN_66.9040-21_MTC
- J2, J4: value 23AH8785-Black -> CONN_66.9040-21_MTC
- PS1, PS2: value IRM-03-15 -> CONV_IRM-03-15
- Q2, Q3, Q4, Q5: value C3M0025065K -> TO-247-4_CRW
- R2: value CW005100R0JE12HE -> RES_CW005_VIS
- U1, U2, U3, U4: value UCC21710QDWRQ1 -> SOIC127P1030X265-16N
- moved G*** 42.6 mm to (68.0, 59.1), turned to 180 degrees
- moved TP2 17.4 mm to (57.0, 65.5)
- moved TP68 16.1 mm to (97.6, 64.2)
- moved R44 16.0 mm to (83.5, 48.0)
- moved C66 15.9 mm to (80.0, 42.2)
- moved D6 15.9 mm to (64.0, 46.6)
- moved D7 15.9 mm to (76.5, 41.8)
- moved F1 15.9 mm to (52.5, 50.6)
- moved J1 15.9 mm to (47.5, 34.2)
- moved J2 15.9 mm to (47.0, 61.2)
- moved J23 15.9 mm to (98.1, 51.1)
- moved R45 15.9 mm to (79.5, 46.8)
- moved R46 15.9 mm to (74.0, 46.8)
- moved R47 15.9 mm to (70.0, 42.8)
- moved TP69 15.9 mm to (97.5, 31.8)
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Routing:
- net /Con_Pro_Gate_node_output: track 0.00 -> 46.5 mm, vias 0 -> 1
- net /EMI_Input_Filter/+VIN_EMI: track 0.00 -> 36.7 mm
- net -VIN: track 0.00 -> 32.7 mm
- net +VIN: track 0.00 -> 30.9 mm
- net GND: track 0.00 -> 18.4 mm, vias 0 -> 9
- net Net-(Q8-G): track 0.00 -> 6.51 mm
- net Net-(R44-Pad2): track 0.00 -> 2.57 mm
- added copper zone on F.Cu, net /EMI_Input_Filter/+VIN_EMI
- added copper zone on B.Cu, net GND
Other:
- board size 322.1 x 269.5 mm -> 392.1 x 268.5 mm
- board text added: "+VIN"
- board text added: "+VIN_Pro"
- board text added: "-VIN"
- board text added: "DC Input / Protection Circuit"
- board text added: "Design By Joseph J. Vitale"
- board text added: "GND"
- board text added: "G_Node"
- board text added: "SiC Single Phase Inverter B1.0"
- board text removed: "DC Input & Input Protection Circuit"

Commit message: WIP PCB Traceing/Layout
Routing:
- net +VIN: track 30.9 -> 0.18 mm
- net -VIN: track 32.7 -> 12.4 mm
- added copper zone on F.Cu, net +VIN
- added copper zone on F.Cu, net -VIN

Commit message: Updating README
Parts:
- added G***: LOGO, SiC_Inverter:Inverter_PCB_Icon, B.Cu at (139.0, 139.0)
- added H5: MountingHole, MountingHole:MountingHole_2.2mm_M2, F.Cu at (170.2, 100.3)
- added H6: MountingHole, MountingHole:MountingHole_2.2mm_M2, F.Cu at (170.2, 153.4)
- added H7: MountingHole, MountingHole:MountingHole_2.2mm_M2, F.Cu at (106.2, 100.3)
- added H8: MountingHole, MountingHole:MountingHole_2.2mm_M2, F.Cu at (106.2, 153.4)
- J1, J3: value CONN_66.9040-21_MTC -> 23AH8786-Red
- J2, J4: value CONN_66.9040-21_MTC -> 23AH8785-Black
- PS1, PS2: value CONV_IRM-03-15 -> IRM-03-15
- Q2, Q3, Q4, Q5: value TO-247-4_CRW -> C3M0025065K
- R2: value RES_CW005_VIS -> CW005100R0JE12HE
- U1, U2, U3, U4: value SOIC127P1030X265-16N -> UCC21710QDWRQ1
- moved J5 499.2 mm to (106.5, 122.0), turned to -90 degrees
- moved J25 482.6 mm to (156.4, 34.1)
- moved J26 482.6 mm to (156.4, 43.3)
- moved J27 482.6 mm to (156.4, 52.4)
- moved PS1 482.6 mm to (123.0, 42.0)
- moved PS2 482.6 mm to (123.0, 67.5)
- moved TP70 482.6 mm to (145.4, 59.8)
- moved TP71 482.6 mm to (145.4, 66.1)
- moved TP72 482.6 mm to (151.6, 59.8)
- moved TP73 482.6 mm to (151.6, 66.1)
- moved TP74 482.6 mm to (157.9, 59.8)
- moved TP75 482.6 mm to (157.9, 66.1)
- moved U5 482.6 mm to (146.4, 72.1)
- moved C1 452.7 mm to (129.2, 117.2), turned to 90 degrees
- moved TP6 435.2 mm to (169.7, 110.9)
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Routing:
- added copper zone on F.Cu, net /EMI_Input_Filter/BUS+_Filtered
- added copper zone on F.Cu, net /EMI_Input_Filter/BUS+_RAW

Commit message: WIP PCB Design
Parts:
- added G***: LOGO, SiC_Inverter:Inverter_PCB_Icon, B.Cu at (223.5, 142.5)
- added G***: LOGO, SiC_Inverter:Inverter_PCB_Icon, B.Cu at (142.4, 62.5)
- added H10: MountingHole, MountingHole:MountingHole_2.2mm_M2, F.Cu at (111.1, 87.6)
- added H11: MountingHole, MountingHole:MountingHole_2.2mm_M2, F.Cu at (184.6, 41.6)
- added H12: MountingHole, MountingHole:MountingHole_2.2mm_M2, F.Cu at (184.4, 87.6)
- added H13: MountingHole, MountingHole:MountingHole_2.2mm_M2, F.Cu at (201.0, 109.5)
- added H14: MountingHole, MountingHole:MountingHole_2.2mm_M2, F.Cu at (246.5, 109.5)
- added H15: MountingHole, MountingHole:MountingHole_2.2mm_M2, F.Cu at (246.0, 145.0)
- added H16: MountingHole, MountingHole:MountingHole_2.2mm_M2, F.Cu at (201.0, 144.5)
- added H9: MountingHole, MountingHole:MountingHole_2.2mm_M2, F.Cu at (111.1, 41.6)
- moved J8 365.5 mm to (200.0, 122.5), turned to -90 degrees
- moved R2 338.7 mm to (206.0, 142.5)
- moved R1 337.8 mm to (214.5, 120.0)
- moved J9 335.5 mm to (247.0, 131.0), turned to 90 degrees
- moved R4 333.1 mm to (220.0, 118.5), turned to 90 degrees
- moved Q1 332.8 mm to (220.1, 129.8), turned to 180 degrees
- moved TP7 331.9 mm to (215.5, 110.1)
- moved D1 330.3 mm to (227.5, 122.0)
- moved J7 320.9 mm to (235.8, 111.5)
- moved R3 320.1 mm to (232.5, 121.5), turned to 90 degrees
- moved TP9 302.4 mm to (246.0, 116.5)
- moved TP8 299.6 mm to (246.0, 138.0)
- moved C65 271.8 mm to (251.0, 82.5)
- moved C68 271.8 mm to (296.5, 66.7)
- moved IC2 271.8 mm to (290.9, 65.4)
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Connections:
- J27 pad 4: +15V_ISO_LBLS -> +15V_ISO_LALS
- PS1 pad 16: +15V_ISO_LBLS -> +15V_ISO_LALS
- TP72 pad 1: +15V_ISO_LBLS -> +15V_ISO_LALS
- U5 pad 1: +15V_ISO_LBLS -> +15V_ISO_LALS
Routing:
- net +15V_ISO_LALS: track 0.00 -> 128.6 mm
- net GND_ISO_LAHS: track 0.00 -> 101.4 mm
- net /Con_Pro_Gate_node_output: track 46.5 -> 133.4 mm
- net GND_ISO_LBHS: track 0.00 -> 58.2 mm
- net +15V_ISO_LBLS: track 0.00 -> 56.5 mm
- net +3V3: track 0.00 -> 39.0 mm
- net LOGIC_GND: track 0.00 -> 27.9 mm
- net /EMI_Input_Filter/+VIN_EMI: track 36.3 -> 35.0 mm
Other:
- board text added: "(325-425) VDC Input"
- board text added: "DC+"
- board text added: "High to Low Voltage Board"
- board text added: "Pre-Charge Circuit"
- board text added: "To Controller"
- board text added: "To Power Board"
