File: Schematics/EMI_Input_Filter.kicad_sch (KiCad schematic)
At the start: 7 parts, among them J5 464379202, J6 464369202

Commit message: Updating README
Parts:
- added H5, H6, H7, H8: MountingHole, MountingHole:MountingHole_2.2mm_M2, symbol Mechanical:MountingHole
