File: Schematics/Sub_PCB_Sheets/Controller_Circuit/Controller_Circuit.kicad_pcb (KiCad board)
At the start: 2 copper layers, 494.6 x 179.4 mm, 277 parts, among them IC1 F280049CPMSR, IC2 CP2102N-A02-GQFN24R, IC3 TPD2EUSB30ADRTR, J1 23AH8786-Red, J10 464379202, J11 464369202, J12 464379202, J13 43045-1212, J14 43650-0418, J15 43650-0418, J16 464369202, J17 464379202, J18 43650-0418, J19 FTSH-105-01-LM-D-K, J2 23AH8785-Black, J20 43045-1212, J21 43650-0418, J22 43650-0418, J23 464369202, J24 43650-0418, J25 43650-0418, J26 43650-0418, J27 43650-0418, J28 1051330011, J3 23AH8786-Red, J4 23AH8785-Black, J5 464379202, J6 464369202, J7 43650-0418, J8 464379202, J9 464369202, Q1 STB10NK60ZT4, Q2 C3M0025065K, Q3 C3M0025065K, Q4 C3M0025065K, Q5 C3M0025065K, Q6 PC817X1CSP9F, Q7 PC817X1CSP9F, Q8 STB10NK60ZT4, U1 UCC21710QDWRQ1, U2 UCC21710QDWRQ1, U3 UCC21710QDWRQ1, U4 UCC21710QDWRQ1, U5 TR05S3V3, Y1 ABM8-20.000MHZ-B2-T

Commit message: updated controller PCB to 4 layer and finished PCB tracing
Parts:
- removed C1: 1 uF, SiC_Inverter:R71PI410050H6K
- removed C10, C12, C14, C15, C16, C2, C3, C4, C6, C8: 22 uF, SiC_Inverter:ESH226M500AL4AA
- removed C11, C13, C5, C7, C9: 2 uF, SiC_Inverter:MKP1848C52050JK2
- removed C17, C18, C35, C36: 15 uF, Capacitor_SMD:C_1206_3216Metric_Pad1.33x1.80mm_HandSolder
- removed C19, C20, C26, C29, C30, C33, C37, C38, C44, C47, C48, C51, C66: 0.1 uF, Capacitor_SMD:C_0805_2012Metric_Pad1.18x1.45mm_HandSolder
- removed C21, C22, C27, C34, C39, C40, C45, C52: 1 uF, Capacitor_SMD:C_1206_3216Metric_Pad1.33x1.80mm_HandSolder
- removed C23, C24, C25, C28, C31, C32, C41, C42, C43, C46, C49, C50: 100 pF, Capacitor_SMD:C_0603_1608Metric_Pad1.08x0.95mm_HandSolder
- removed C53: 6.8 uF, SiC_Inverter:C4AF9BW4680T3FK
- removed D1, D7: BZX84C15-7-F, Package_TO_SOT_SMD:SOT-23-3
- removed D2, D3, D4, D5: BZX84C20-7-F, Package_TO_SOT_SMD:SOT-23-3
- removed D6: P6KE500A-HF, Diode_THT:D_DO-15_P12.70mm_Horizontal
- removed F1: 0031.8322, SiC_Inverter:0031.8322
- removed the G*** at (500.1, 162.0)
- removed the G*** at (67.5, 176.0)
- removed the G*** at (153.3, 177.6)
- removed the G*** at (299.4, 164.9)
- removed the G*** at (224.0, 180.9)
- removed the G*** at (382.6, 134.4)
- removed the G*** at (142.9, 100.9)
- removed H1, H10, H11, H12, H13, H14, H15, H16, H17, H18, H19, H2, H20, H25, H26, H27, H28, H29, H3, H30, H31, H32, H4, H5, H6, H7, H8, H9: MountingHole, MountingHole:MountingHole_2.2mm_M2
- removed IC3: TPD2EUSB30ADRTR, SiC_Inverter:TPD2EUSB30ADRTR
- removed J1, J3: 23AH8786-Red, SiC_Inverter:23AH8786-Red
- removed J10, J12, J17, J5, J8: 464379202, SiC_Inverter:46437-900_02
- removed J11, J16, J23, J6, J9: 464369202, SiC_Inverter:46436-900_02
- removed J13: 43045-1212, SiC_Inverter:43045-1212
- removed J14, J15, J24, J25, J26, J27, J7: 43650-0418, SiC_Inverter:436500418
- removed J2, J4: 23AH8785-Black, SiC_Inverter:23AH8785-Black
- removed L1: 47 uH, SiC_Inverter:2300HT_470
- removed L2: 2.2 mH, SiC_Inverter:7448258022
- removed L3, L4: 470 uH, SiC_Inverter:1140471KRC
- removed PS1, PS2: IRM-03-15, SiC_Inverter:IRM-03-15
- removed Q1, Q8: STB10NK60ZT4, Package_TO_SOT_SMD:TO-263-2
- removed Q2, Q3, Q4, Q5: C3M0025065K, SiC_Inverter:C3M0025065K
- removed R1, R44, R45: 499 K, Resistor_SMD:R_1206_3216Metric_Pad1.30x1.75mm_HandSolder
- removed R10, R21, R22, R23, R24, R7, R8, R9: 10, Resistor_SMD:R_1206_3216Metric_Pad1.30x1.75mm_HandSolder
- removed R11, R13, R14, R16, R17, R18, R25, R27, R28, R30, R31, R32: 5 K, Resistor_SMD:R_1206_3216Metric_Pad1.30x1.75mm_HandSolder
- removed R12, R15, R26, R29: 100, Resistor_SMD:R_1206_3216Metric_Pad1.30x1.75mm_HandSolder
- removed R19, R20, R4, R47, R5, R6: 100 K, Resistor_SMD:R_1206_3216Metric_Pad1.30x1.75mm_HandSolder
- removed R2: CW005100R0JE12HE, SiC_Inverter:CW005100R0JE12HE
- removed R3, R46: 47, Resistor_SMD:R_1206_3216Metric_Pad1.30x1.75mm_HandSolder
- removed R33: 6, SiC_Inverter:CW005100R0JE12HE
- removed TP1, TP11, TP24, TP25, TP26, TP27, TP3, TP32, TP34, TP35, TP36, TP37, TP5, TP67, TP69, TP7, TP71, TP72, TP74, TP8: 5277, SiC_Inverter:5277
- removed TP10, TP2, TP33, TP4, TP6, TP68, TP70, TP73, TP75, TP9: 5281, SiC_Inverter:5281
- removed U1, U2, U3, U4: UCC21710QDWRQ1, SiC_Inverter:UCC21710QDWRQ1
- removed U5: TR05S3V3, SiC_Inverter:TR05S3V3
- moved J28 139.5 mm to (140.1, 85.8), turned to 90 degrees
- moved C69 138.7 mm to (138.5, 93.2), turned to -90 degrees
- moved R34 137.3 mm to (134.9, 92.9), turned to 180 degrees
- moved C54 136.0 mm to (114.8, 99.7)
- moved C55 136.0 mm to (114.8, 97.7)
- moved C56 136.0 mm to (114.8, 101.7)
- moved C63 136.0 mm to (114.8, 95.7)
- moved H23 136.0 mm to (92.3, 77.7)
- moved TP45 136.0 mm to (153.4, 96.0)
- moved TP50 136.0 mm to (147.1, 96.0)
- moved TP63 136.0 mm to (135.2, 122.7)
- moved Y1 136.0 mm to (121.5, 112.0)
- moved C57 136.0 mm to (126.9, 110.9)
- moved C58 136.0 mm to (128.9, 110.9)
- moved C64 136.0 mm to (118.0, 111.8)
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Routing:
- net +15V_ISO_LALS: track 150.9 -> 0.00 mm
- net LOGIC_GND: track 232.6 -> 81.7 mm, vias 36 -> 23
- net GND_ISO_LAHS: track 137.6 -> 0.00 mm, vias 6 -> 0
- net /Con_Pro_Gate_node_output: track 154.7 -> 21.3 mm, vias 1 -> 0
- net GND: track 192.5 -> 77.3 mm, vias 24 -> 2
- net +3V3: track 194.4 -> 103.9 mm, vias 32 -> 25
- net GND_ISO_LBHS: track 88.2 -> 0.00 mm, vias 10 -> 0
- net +15V_ISO_LBLS: track 81.2 -> 0.00 mm
- net /Con_EN_A_H: track 49.2 -> 96.4 mm, vias 0 -> 1
- net /Full-Bridge/Leg_A_Power_Stage/LegA_LS_Gate: track 44.6 -> 0.00 mm
- net /Full-Bridge/Leg_A_Power_Stage/LegA_HS_Gate: track 44.1 -> 0.00 mm
- net /Full-Bridge/Leg_B_Power_Stage/LegB_LS_Gate: track 38.6 -> 0.00 mm
- net /Con_Gate_node_prech: track 67.4 -> 29.1 mm
- net /Con_FLT_A_H: track 45.8 -> 82.7 mm, vias 0 -> 1
- net /Full-Bridge/Leg_B_Power_Stage/LegB_HS_Gate: track 35.9 -> 0.00 mm
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- added copper zone on In2.Cu, net +3V3
- added copper zone on In1.Cu, net LOGIC_GND
- removed copper zone on B.Cu, net +3V3
- removed copper zone on F.Cu, net +VIN
- removed copper zone on F.Cu, net -VIN
- removed copper zone on F.Cu, net /DC_Link_Caps/BUS_DC+
- removed copper zone on F.Cu, net /EMI_Input_Filter/+VIN_EMI
- removed copper zone on F.Cu, net /EMI_Input_Filter/BUS+_Filtered
- removed copper zone on F.Cu, net /EMI_Input_Filter/BUS+_RAW
- removed copper zone on F.Cu, net /Phase_A_Output
- removed copper zone on B.Cu, net /Phase_B_Output
- removed copper zone on B.Cu, net GND
- removed copper zone on B.Cu, net GND_ISO_LAHS
- removed copper zone on F.Cu, net GND_ISO_LBHS
- removed copper zone on B.Cu, net LOGIC_GND
Other:
- board size 494.6 x 179.4 mm -> 109.6 x 62.6 mm
- copper layers 2 -> 4
- board text removed: "(325-425) VDC Input"
- board text removed: "+15VDC"
- board text removed: "+DC Filtered"
- board text removed: "+DC_BUS"
- board text removed: "+VIN"
- board text removed: "+VIN_Pro"
- board text removed: "-VIN"
- board text removed: "120Vrms Single Phase L-L"
- board text removed: "2.08 Inches"
- board text removed: "AC Output Filter"
- board text removed: "DC Input / Protection Circuit"
- board text removed: "DC Input and Input Protection Circuit"
- board text removed: "DC Link Caps"
- board text removed: "DC+"
- board text removed: "EMI Input Filter"
- board text removed: "Full-Bridge"
- board text removed: "G_Node"
- board text removed: "HS_Gate"
- board text removed: "High Side"
- board text removed: "High to Low Voltage Board"
- board text removed: "ISO_GND"
- board text removed: "LAHS"
- board text removed: "LALS"
- board text removed: "LBHS"
- board text removed: "LBLS"
- board text removed: "LS_Gate"
- board text removed: "Leg A"
- board text removed: "Leg B"
- board text removed: "Low Side"
- board text removed: "Need to move to a 4 layer board when on its own PCB sheet"
- board text removed: "PWM_A_H"
- board text removed: "PWM_A_L"
- board text removed: "PWM_B_H"
- board text removed: "PWM_B_L"
- board text removed: "Phase A Node"
- board text removed: "Phase A Output"
- board text removed: "Phase B Node"
- board text removed: "Phase B Output"
- board text removed: "Power"
- board text removed: "Pre-Charge Circuit"
- board text removed: "Pre-Charge_Current_Limiting"
- board text removed: "SiC Full Bridge"
- board text removed: "To Controller J18"
- board text removed: "To Controller J20"
- board text removed: "To Controller J21"
- board text removed: "To Controller J22"
- board text removed: "To DC Input J24"
- board text removed: "To Full-Bridge J15"
- board text removed: "To Power Board J25"
- board text removed: "To Power J27"
