File: Schematics/Sub_PCB_Sheets/DC_Link_Caps/DC_Link_Caps_Circuit.kicad_pcb (KiCad board)
At the start: 2 copper layers, 494.6 x 179.4 mm, 277 parts, among them IC1 F280049CPMSR, IC2 CP2102N-A02-GQFN24R, IC3 TPD2EUSB30ADRTR, J1 23AH8786-Red, J10 464379202, J11 464369202, J12 464379202, J13 43045-1212, J14 43650-0418, J15 43650-0418, J16 464369202, J17 464379202, J18 43650-0418, J19 FTSH-105-01-LM-D-K, J2 23AH8785-Black, J20 43045-1212, J21 43650-0418, J22 43650-0418, J23 464369202, J24 43650-0418, J25 43650-0418, J26 43650-0418, J27 43650-0418, J28 1051330011, J3 23AH8786-Red, J4 23AH8785-Black, J5 464379202, J6 464369202, J7 43650-0418, J8 464379202, J9 464369202, Q1 STB10NK60ZT4, Q2 C3M0025065K, Q3 C3M0025065K, Q4 C3M0025065K, Q5 C3M0025065K, Q6 PC817X1CSP9F, Q7 PC817X1CSP9F, Q8 STB10NK60ZT4, U1 UCC21710QDWRQ1, U2 UCC21710QDWRQ1, U3 UCC21710QDWRQ1, U4 UCC21710QDWRQ1, U5 TR05S3V3, Y1 ABM8-20.000MHZ-B2-T

Commit message: Finishing the DC Link Caps and Fab Outputs
Parts:
- removed C1: 1 uF, SiC_Inverter:R71PI410050H6K
- removed C17, C18, C35, C36: 15 uF, Capacitor_SMD:C_1206_3216Metric_Pad1.33x1.80mm_HandSolder
- removed C19, C20, C26, C29, C30, C33, C37, C38, C44, C47, C48, C51, C54, C55, C56, C57, C58, C60, C61, C62, C63, C66, C67: 0.1 uF, Capacitor_SMD:C_0805_2012Metric_Pad1.18x1.45mm_HandSolder
- removed C21, C22, C27, C34, C39, C40, C45, C52, C69: 1 uF, Capacitor_SMD:C_1206_3216Metric_Pad1.33x1.80mm_HandSolder
- removed C23, C24, C25, C28, C31, C32, C41, C42, C43, C46, C49, C50: 100 pF, Capacitor_SMD:C_0603_1608Metric_Pad1.08x0.95mm_HandSolder
- removed C53: 6.8 uF, SiC_Inverter:C4AF9BW4680T3FK
- removed C59, C68: 10 uF, Capacitor_SMD:C_0805_2012Metric_Pad1.18x1.45mm_HandSolder
- removed C64, C65: 18 pF, Capacitor_SMD:C_0402_1005Metric_Pad0.74x0.62mm_HandSolder
- removed D1, D7: BZX84C15-7-F, Package_TO_SOT_SMD:SOT-23-3
- removed D2, D3, D4, D5: BZX84C20-7-F, Package_TO_SOT_SMD:SOT-23-3
- removed D6: P6KE500A-HF, Diode_THT:D_DO-15_P12.70mm_Horizontal
- removed F1: 0031.8322, SiC_Inverter:0031.8322
- removed the G*** at (500.1, 162.0)
- removed the G*** at (67.5, 176.0)
- removed the G*** at (153.3, 177.6)
- removed the G*** at (224.0, 180.9)
- removed the G*** at (382.6, 134.4)
- removed the G*** at (299.1, 62.0)
- removed the G*** at (142.9, 100.9)
- removed H1, H10, H11, H12, H13, H14, H15, H16, H2, H21, H22, H23, H24, H25, H26, H27, H28, H29, H3, H30, H31, H32, H4, H5, H6, H7, H8, H9: MountingHole, MountingHole:MountingHole_2.2mm_M2
- removed IC1: F280049CPMSR, SiC_Inverter:F280049CPMSR
- removed IC2: CP2102N-A02-GQFN24R, SiC_Inverter:CP2102N-A02-GQFN24R
- removed IC3: TPD2EUSB30ADRTR, SiC_Inverter:TPD2EUSB30ADRTR
- removed J1, J3: 23AH8786-Red, SiC_Inverter:23AH8786-Red
- removed J12, J17, J5, J8: 464379202, SiC_Inverter:46437-900_02
- removed J13, J20: 43045-1212, SiC_Inverter:43045-1212
- removed J14, J15, J18, J21, J22, J24, J25, J26, J27, J7: 43650-0418, SiC_Inverter:436500418
- removed J16, J23, J6, J9: 464369202, SiC_Inverter:46436-900_02
- removed J19: FTSH-105-01-LM-D-K, SiC_Inverter:FTSH-105-01-LM-D-K
- removed J2, J4: 23AH8785-Black, SiC_Inverter:23AH8785-Black
- removed J28: 1051330011, SiC_Inverter:105133-0011
- removed L1: 47 uH, SiC_Inverter:2300HT_470
- removed L2: 2.2 mH, SiC_Inverter:7448258022
- removed L3, L4: 470 uH, SiC_Inverter:1140471KRC
- removed PS1, PS2: IRM-03-15, SiC_Inverter:IRM-03-15
- removed Q1, Q8: STB10NK60ZT4, Package_TO_SOT_SMD:TO-263-2
- removed Q2, Q3, Q4, Q5: C3M0025065K, SiC_Inverter:C3M0025065K
- removed Q6, Q7: PC817X1CSP9F, SiC_Inverter:PC817X1CSP9F
- removed R1, R44, R45: 499 K, Resistor_SMD:R_1206_3216Metric_Pad1.30x1.75mm_HandSolder
- removed R10, R21, R22, R23, R24, R7, R8, R9: 10, Resistor_SMD:R_1206_3216Metric_Pad1.30x1.75mm_HandSolder
- removed R11, R13, R14, R16, R17, R18, R25, R27, R28, R30, R31, R32: 5 K, Resistor_SMD:R_1206_3216Metric_Pad1.30x1.75mm_HandSolder
- removed R12, R15, R26, R29: 100, Resistor_SMD:R_1206_3216Metric_Pad1.30x1.75mm_HandSolder
- removed R19, R20, R34, R36, R37, R39, R4, R40, R41, R43, R47, R48, R5, R6: 100 K, Resistor_SMD:R_1206_3216Metric_Pad1.30x1.75mm_HandSolder
- removed R2: CW005100R0JE12HE, SiC_Inverter:CW005100R0JE12HE
- removed R3, R46: 47, Resistor_SMD:R_1206_3216Metric_Pad1.30x1.75mm_HandSolder
- removed R33: 6, SiC_Inverter:CW005100R0JE12HE
- removed R35, R42: 10 K, Resistor_SMD:R_1206_3216Metric_Pad1.30x1.75mm_HandSolder
- removed R38: 2 K, Resistor_SMD:R_1206_3216Metric_Pad1.30x1.75mm_HandSolder
- removed R49: 0, Resistor_SMD:R_1206_3216Metric_Pad1.30x1.75mm_HandSolder
- removed TP1, TP24, TP25, TP26, TP27, TP3, TP32, TP34, TP35, TP36, TP37, TP38, TP40, TP41, TP42, TP43, TP44, TP45, TP46, TP47, TP48, TP49, TP5, TP50, TP51, TP52, TP53, TP54, TP55, TP56, TP57, TP58, TP60, TP61, TP62, TP63, TP64, TP65, TP67, TP69, TP7, TP71, TP72, TP74, TP8: 5277, SiC_Inverter:5277
- removed TP2, TP33, TP39, TP4, TP59, TP6, TP66, TP68, TP70, TP73, TP75, TP76, TP9: 5281, SiC_Inverter:5281
- removed U1, U2, U3, U4: UCC21710QDWRQ1, SiC_Inverter:UCC21710QDWRQ1
- removed U5: TR05S3V3, SiC_Inverter:TR05S3V3
- removed Y1: ABM8-20.000MHZ-B2-T, SiC_Inverter:ABM8-20.000MHZ-B2-T
- moved TP11 22.6 mm to (317.0, 124.2)
- moved TP10 22.5 mm to (317.0, 146.8)
- moved H17 7.25 mm to (265.2, 212.2)
- moved H18 6.93 mm to (265.6, 119.0)
- moved H19 4.28 mm to (318.8, 118.8)
- moved H20 4.20 mm to (318.7, 212.4)
- moved J10 1.45 mm to (265.4, 160.9)
Routing:
- net LOGIC_GND: track 232.6 -> 0.00 mm, vias 36 -> 0
- net +3V3: track 194.4 -> 0.00 mm, vias 32 -> 0
- net GND: track 192.5 -> 0.00 mm, vias 24 -> 0
- net /Con_Pro_Gate_node_output: track 154.7 -> 0.00 mm, vias 1 -> 0
- net +15V_ISO_LALS: track 150.9 -> 0.00 mm
- net GND_ISO_LAHS: track 137.6 -> 0.00 mm, vias 6 -> 0
- net /Con_PWM_A_H: track 116.7 -> 0.00 mm, vias 1 -> 0
- net /Con_PWM_A_L: track 104.9 -> 0.00 mm, vias 1 -> 0
- net /Con_EN_B_H: track 104.7 -> 0.00 mm, vias 1 -> 0
- net /Con_PWM_B_H: track 97.3 -> 0.00 mm, vias 1 -> 0
- net /Con_PWM_B_L: track 92.3 -> 0.00 mm, vias 1 -> 0
- net /Con_EN_A_L: track 91.9 -> 0.00 mm, vias 1 -> 0
- net /Con_FLT_B_H: track 88.3 -> 0.00 mm, vias 1 -> 0
- net GND_ISO_LBHS: track 88.2 -> 0.00 mm, vias 10 -> 0
- net /Con_RDY_A_H: track 85.5 -> 0.00 mm, vias 1 -> 0
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- removed copper zone on B.Cu, net +3V3
- removed copper zone on F.Cu, net +VIN
- removed copper zone on F.Cu, net -VIN
- removed copper zone on F.Cu, net /EMI_Input_Filter/+VIN_EMI
- removed copper zone on F.Cu, net /EMI_Input_Filter/BUS+_Filtered
- removed copper zone on F.Cu, net /EMI_Input_Filter/BUS+_RAW
- removed copper zone on F.Cu, net /Phase_A_Output
- removed copper zone on B.Cu, net /Phase_B_Output
- removed copper zone on B.Cu, net GND_ISO_LAHS
- removed copper zone on F.Cu, net GND_ISO_LBHS
- removed copper zone on B.Cu, net LOGIC_GND
Other:
- board size 494.6 x 179.4 mm -> 62.5 x 100.5 mm
- board text removed: "(325-425) VDC Input"
- board text removed: "+15VDC"
- board text removed: "+3V3"
- board text removed: "+DC Filtered"
- board text removed: "+VIN"
- board text removed: "+VIN_Pro"
- board text removed: "-VIN"
- board text removed: "120Vrms Single Phase L-L"
- board text removed: "2.08 Inches"
- board text removed: "AC Output Filter"
- board text removed: "CPro G_Node"
- board text removed: "Controller + USB"
- board text removed: "DC Input / Protection Circuit"
- board text removed: "DC Input and Input Protection Circuit"
- board text removed: "DC+"
- board text removed: "EMI Input Filter"
- board text removed: "EN_AH"
- board text removed: "EN_AL"
- board text removed: "EN_BH"
- board text removed: "EN_BL"
- board text removed: "FLT_AH"
- board text removed: "FLT_AL"
- board text removed: "FLT_BH"
- board text removed: "FLT_BL"
- board text removed: "Full-Bridge"
- board text removed: "G_Node"
- board text removed: "HS_Gate"
- board text removed: "High Side"
- board text removed: "High to Low Voltage Board"
- board text removed: "ISO_GND"
- board text removed: "J-TAG"
- board text removed: "LAHS"
- board text removed: "LALS"
- board text removed: "LBHS"
- board text removed: "LBLS"
- board text removed: "LS_Gate"
- board text removed: "L_GND"
- board text removed: "Leg A"
- board text removed: "Leg B"
- board text removed: "Logic GND"
- board text removed: "Low Side"
- board text removed: "Need to move to a 4 layer board when on its own PCB sheet"
- board text removed: "Open Loop Design"
- board text removed: "PWM AH"
- board text removed: "PWM AL"
- board text removed: "PWM BH"
- board text removed: "PWM BL"
- board text removed: "PWM_A_H"
- board text removed: "PWM_A_L"
- board text removed: "PWM_B_H"
- board text removed: "PWM_B_L"
- board text removed: "Phase A Node"
- board text removed: "Phase A Output"
- board text removed: "Phase B Node"
- board text removed: "Phase B Output"
- board text removed: "Power"
- board text removed: "Pre G_Node"
- board text removed: "Pre-Charge Circuit"
- board text removed: "Pre-Charge_Current_Limiting"
- board text removed: "Pro G_Node"
- board text removed: "RDY_AH"
- board text removed: "RDY_AL"
- board text removed: "RDY_BH"
- board text removed: "RDY_BL"
- board text removed: "SiC Full Bridge"
- board text removed: "SiC Single Phase Inverter Controller"
- board text removed: "TCK"
- board text removed: "TDI"
- board text removed: "TDO"
- board text removed: "TMS"
- board text removed: "To Controller J18"
- board text removed: "To Controller J20"
- board text removed: "To Controller J21"
- board text removed: "To Controller J22"
- board text removed: "To DC Input J24"
- board text removed: "To Full-Bridge J13"
- board text removed: "To Full-Bridge J14"
- board text removed: "To Full-Bridge J15"
- board text removed: "To Power Board J25"
- board text removed: "To Power J26"
- board text removed: "To Power J27"
- board text removed: "To Pre-Charge J7"
- board text removed: "X1"
- board text removed: "X2"
- board text removed: "XRS"
