File: Schematics/Sub_PCB_Sheets/Full-Bridge/Full_Bridge_Circuit.kicad_pcb (KiCad board)
At the start: 2 copper layers, 494.6 x 179.4 mm, 277 parts, among them IC1 F280049CPMSR, IC2 CP2102N-A02-GQFN24R, IC3 TPD2EUSB30ADRTR, J1 23AH8786-Red, J10 464379202, J11 464369202, J12 464379202, J13 43045-1212, J14 43650-0418, J15 43650-0418, J16 464369202, J17 464379202, J18 43650-0418, J19 FTSH-105-01-LM-D-K, J2 23AH8785-Black, J20 43045-1212, J21 43650-0418, J22 43650-0418, J23 464369202, J24 43650-0418, J25 43650-0418, J26 43650-0418, J27 43650-0418, J28 1051330011, J3 23AH8786-Red, J4 23AH8785-Black, J5 464379202, J6 464369202, J7 43650-0418, J8 464379202, J9 464369202, Q1 STB10NK60ZT4, Q2 C3M0025065K, Q3 C3M0025065K, Q4 C3M0025065K, Q5 C3M0025065K, Q6 PC817X1CSP9F, Q7 PC817X1CSP9F, Q8 STB10NK60ZT4, U1 UCC21710QDWRQ1, U2 UCC21710QDWRQ1, U3 UCC21710QDWRQ1, U4 UCC21710QDWRQ1, U5 TR05S3V3, Y1 ABM8-20.000MHZ-B2-T

Commit message: Adding two pin connector for 3V3 from power to Full-Bridge
Parts:
- removed C1: 1 uF, SiC_Inverter:R71PI410050H6K
- removed C10, C12, C14, C15, C16, C2, C3, C4, C6, C8: 22 uF, SiC_Inverter:ESH226M500AL4AA
- removed C11, C13, C5, C7, C9: 2 uF, SiC_Inverter:MKP1848C52050JK2
- removed C53: 6.8 uF, SiC_Inverter:C4AF9BW4680T3FK
- removed C54, C55, C56, C57, C58, C60, C61, C62, C63, C66, C67: 0.1 uF, Capacitor_SMD:C_0805_2012Metric_Pad1.18x1.45mm_HandSolder
- removed C59, C68: 10 uF, Capacitor_SMD:C_0805_2012Metric_Pad1.18x1.45mm_HandSolder
- removed C64, C65: 18 pF, Capacitor_SMD:C_0402_1005Metric_Pad0.74x0.62mm_HandSolder
- removed C69: 1 uF, Capacitor_SMD:C_1206_3216Metric_Pad1.33x1.80mm_HandSolder
- removed D1, D7: BZX84C15-7-F, Package_TO_SOT_SMD:SOT-23-3
- removed D6: P6KE500A-HF, Diode_THT:D_DO-15_P12.70mm_Horizontal
- removed F1: 0031.8322, SiC_Inverter:0031.8322
- removed the G*** at (500.1, 162.0)
- removed the G*** at (67.5, 176.0)
- removed the G*** at (153.3, 177.6)
- removed the G*** at (299.4, 164.9)
- removed the G*** at (224.0, 180.9)
- removed the G*** at (299.1, 62.0)
- removed the G*** at (142.9, 100.9)
- removed H1, H10, H11, H12, H13, H14, H15, H16, H17, H18, H19, H2, H20, H21, H22, H23, H24, H29, H3, H30, H31, H32, H4, H5, H6, H7, H8, H9: MountingHole, MountingHole:MountingHole_2.2mm_M2
- removed IC1: F280049CPMSR, SiC_Inverter:F280049CPMSR
- removed IC2: CP2102N-A02-GQFN24R, SiC_Inverter:CP2102N-A02-GQFN24R
- removed IC3: TPD2EUSB30ADRTR, SiC_Inverter:TPD2EUSB30ADRTR
- removed J1, J3: 23AH8786-Red, SiC_Inverter:23AH8786-Red
- removed J10, J17, J5, J8: 464379202, SiC_Inverter:46437-900_02
- removed J11, J23, J6, J9: 464369202, SiC_Inverter:46436-900_02
- removed J18, J21, J22, J24, J25, J26, J27, J7: 43650-0418, SiC_Inverter:436500418
- removed J19: FTSH-105-01-LM-D-K, SiC_Inverter:FTSH-105-01-LM-D-K
- removed J2, J4: 23AH8785-Black, SiC_Inverter:23AH8785-Black
- removed J20: 43045-1212, SiC_Inverter:43045-1212
- removed J28: 1051330011, SiC_Inverter:105133-0011
- removed L1: 47 uH, SiC_Inverter:2300HT_470
- removed L2: 2.2 mH, SiC_Inverter:7448258022
- removed L3, L4: 470 uH, SiC_Inverter:1140471KRC
- removed PS1, PS2: IRM-03-15, SiC_Inverter:IRM-03-15
- removed Q1, Q8: STB10NK60ZT4, Package_TO_SOT_SMD:TO-263-2
- removed Q6, Q7: PC817X1CSP9F, SiC_Inverter:PC817X1CSP9F
- removed R1, R44, R45: 499 K, Resistor_SMD:R_1206_3216Metric_Pad1.30x1.75mm_HandSolder
- removed R2: CW005100R0JE12HE, SiC_Inverter:CW005100R0JE12HE
- removed R3, R46: 47, Resistor_SMD:R_1206_3216Metric_Pad1.30x1.75mm_HandSolder
- removed R33: 6, SiC_Inverter:CW005100R0JE12HE
- removed R34, R36, R37, R39, R4, R40, R41, R43, R47, R48: 100 K, Resistor_SMD:R_1206_3216Metric_Pad1.30x1.75mm_HandSolder
- removed R35, R42: 10 K, Resistor_SMD:R_1206_3216Metric_Pad1.30x1.75mm_HandSolder
- removed R38: 2 K, Resistor_SMD:R_1206_3216Metric_Pad1.30x1.75mm_HandSolder
- removed R49: 0, Resistor_SMD:R_1206_3216Metric_Pad1.30x1.75mm_HandSolder
- removed TP1, TP11, TP3, TP38, TP40, TP41, TP42, TP43, TP44, TP45, TP46, TP47, TP48, TP49, TP5, TP50, TP51, TP52, TP53, TP54, TP55, TP56, TP57, TP58, TP60, TP61, TP62, TP63, TP64, TP65, TP67, TP69, TP7, TP71, TP72, TP74, TP8: 5277, SiC_Inverter:5277
- removed TP10, TP2, TP39, TP4, TP59, TP6, TP66, TP68, TP70, TP73, TP75, TP76, TP9: 5281, SiC_Inverter:5281
- removed U5: TR05S3V3, SiC_Inverter:TR05S3V3
- removed Y1: ABM8-20.000MHZ-B2-T, SiC_Inverter:ABM8-20.000MHZ-B2-T
- Q2, Q3, Q4, Q5: value C3M0025065K -> TO-247-4_CRW
- U1, U2, U3, U4: value UCC21710QDWRQ1 -> SOIC127P1030X265-16N
- moved J14 251.5 mm to (107.7, 51.7)
- moved C22 244.7 mm to (152.6, 113.5)
- moved C42 244.6 mm to (153.0, 55.2)
- moved D4 244.6 mm to (133.3, 81.5)
- moved R22 244.6 mm to (129.8, 73.7)
- moved TP35 244.6 mm to (167.0, 107.7)
- moved C21 244.6 mm to (125.4, 113.0)
- moved C26 244.6 mm to (157.4, 132.3)
- moved C29 244.6 mm to (148.7, 132.2)
- moved C30 244.6 mm to (122.2, 132.0)
- moved C37 244.6 mm to (120.5, 73.2)
- moved C48 244.6 mm to (131.9, 54.8)
- moved C49 244.6 mm to (127.7, 55.0)
- moved C50 244.6 mm to (125.6, 55.2)
- moved C51 244.6 mm to (121.2, 54.9)
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Routing:
- net LOGIC_GND: track 232.6 -> 57.7 mm, vias 36 -> 25
- net /Con_Pro_Gate_node_output: track 154.7 -> 0.00 mm, vias 1 -> 0
- net +3V3: track 194.4 -> 47.9 mm, vias 32 -> 13
- net GND: track 192.5 -> 52.8 mm, vias 24 -> 19
- net +15V_ISO_LALS: track 150.9 -> 17.4 mm
- net /Con_PWM_A_H: track 116.7 -> 10.5 mm, vias 1 -> 0
- net GND_ISO_LAHS: track 137.6 -> 34.1 mm, vias 6 -> 8
- net /Con_PWM_A_L: track 104.9 -> 10.0 mm, vias 1 -> 0
- net /Con_EN_B_H: track 104.7 -> 11.1 mm, vias 1 -> 0
- net /Con_PWM_B_H: track 97.3 -> 11.2 mm, vias 1 -> 0
- net /Con_PWM_B_L: track 92.3 -> 10.9 mm, vias 1 -> 0
- net /Con_EN_A_L: track 91.9 -> 12.1 mm, vias 1 -> 0
- net /Con_FLT_B_H: track 88.3 -> 11.3 mm, vias 1 -> 0
- net /Con_RDY_A_H: track 85.5 -> 11.3 mm, vias 1 -> 0
- net /Con_FLT_B_L: track 81.8 -> 11.2 mm, vias 1 -> 0
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- added copper zone on In1.Cu, net GND
- added copper zone on B.Cu, net GND_ISO_LBHS
- added copper zone on In1.Cu, net LOGIC_GND
- removed copper zone on B.Cu, net +3V3
- removed copper zone on F.Cu, net +VIN
- removed copper zone on F.Cu, net -VIN
- removed copper zone on F.Cu, net /EMI_Input_Filter/+VIN_EMI
- removed copper zone on F.Cu, net /EMI_Input_Filter/BUS+_Filtered
- removed copper zone on F.Cu, net /EMI_Input_Filter/BUS+_RAW
- removed copper zone on F.Cu, net /Phase_A_Output
- removed copper zone on B.Cu, net /Phase_B_Output
- removed copper zone on B.Cu, net GND
- removed copper zone on F.Cu, net GND_ISO_LBHS
- removed copper zone on B.Cu, net LOGIC_GND
Other:
- board size 494.6 x 179.4 mm -> 85.5 x 108.4 mm
- copper layers 2 -> 4
- board text removed: "(325-425) VDC Input"
- board text removed: "+15VDC"
- board text removed: "+3V3"
- board text removed: "+DC Filtered"
- board text removed: "+DC_BUS"
- board text removed: "+VIN"
- board text removed: "+VIN_Pro"
- board text removed: "-VIN"
- board text removed: "120Vrms Single Phase L-L"
- board text removed: "2.08 Inches"
- board text removed: "AC Output Filter"
- board text removed: "CPro G_Node"
- board text removed: "Controller + USB"
- board text removed: "DC Input / Protection Circuit"
- board text removed: "DC Input and Input Protection Circuit"
- board text removed: "DC Link Caps"
- board text removed: "DC+"
- board text removed: "EMI Input Filter"
- board text removed: "EN_AH"
- board text removed: "EN_AL"
- board text removed: "EN_BH"
- board text removed: "EN_BL"
- board text removed: "FLT_AH"
- board text removed: "FLT_AL"
- board text removed: "FLT_BH"
- board text removed: "FLT_BL"
- board text removed: "GND"
- board text removed: "G_Node"
- board text removed: "High to Low Voltage Board"
- board text removed: "ISO_GND"
- board text removed: "J-TAG"
- board text removed: "LAHS"
- board text removed: "LALS"
- board text removed: "LBHS"
- board text removed: "LBLS"
- board text removed: "L_GND"
- board text removed: "Logic GND"
- board text removed: "Need to move to a 4 layer board when on its own PCB sheet"
- board text removed: "Open Loop Design"
- board text removed: "PWM AH"
- board text removed: "PWM AL"
- board text removed: "PWM BH"
- board text removed: "PWM BL"
- board text removed: "Phase A Output"
- board text removed: "Phase B Output"
- board text removed: "Power"
- board text removed: "Pre G_Node"
- board text removed: "Pre-Charge Circuit"
- board text removed: "Pre-Charge_Current_Limiting"
- board text removed: "Pro G_Node"
- board text removed: "RDY_AH"
- board text removed: "RDY_AL"
- board text removed: "RDY_BH"
- board text removed: "RDY_BL"
- board text removed: "SiC Single Phase Inverter Controller"
- board text removed: "TCK"
- board text removed: "TDI"
- board text removed: "TDO"
- board text removed: "TMS"
- board text removed: "To Controller J18"
- board text removed: "To Controller J22"
- board text removed: "To DC Input J24"
- board text removed: "To Full-Bridge J13"
- board text removed: "To Full-Bridge J14"
- board text removed: "To Full-Bridge J15"
- board text removed: "To Power Board J25"
- board text removed: "To Power J26"
- board text removed: "To Pre-Charge J7"
- board text removed: "X1"
- board text removed: "X2"
- board text removed: "XRS"

Commit message: WIP Full-Bridge PCB tracing
Parts:
- added J29: 43045-0212, SiC_Inverter:43045-0212, F.Cu at (176.1, 53.4)
- moved J14 9.06 mm to (107.7, 60.8), turned to -90 degrees
- moved J13 0.08 mm to (106.2, 128.9)
Routing:
- net /Con_PWM_A_L: track 10.0 -> 133.8 mm, vias 0 -> 1
- net /Con_PWM_A_H: track 10.5 -> 106.9 mm, vias 0 -> 1
- net /Con_EN_A_L: track 12.1 -> 86.5 mm, vias 0 -> 1
- net /Con_FLT_A_L: track 12.3 -> 78.9 mm, vias 0 -> 1
- net /Con_PWM_B_L: track 10.9 -> 69.7 mm, vias 0 -> 1
- net /Con_RDY_A_L: track 11.8 -> 70.5 mm, vias 0 -> 1
- net /Con_EN_A_H: track 11.9 -> 57.3 mm, vias 0 -> 1
- net /Con_FLT_A_H: track 11.3 -> 48.9 mm, vias 0 -> 1
- net /Con_PWM_B_H: track 11.2 -> 42.8 mm, vias 0 -> 1
- net /Con_RDY_A_H: track 11.3 -> 40.5 mm, vias 0 -> 1
- net +15V_ISO_LBLS: track 24.2 -> 15.7 mm, vias 0 -> 4
- net +15V_ISO_LALS: track 17.4 -> 14.5 mm, vias 0 -> 4
- net +3V3: track 47.9 -> 45.9 mm, vias 13 -> 20
- net /Con_RDY_B_H: vias 0 -> 1
- net /Con_RDY_B_L: vias 0 -> 1
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- added copper zone on In2.Cu, net +15V_ISO_LALS
- added copper zone on In2.Cu, net +15V_ISO_LBLS
- added copper zone on In2.Cu, net +3V3
Other:
- board text added: "To Power J30"

Commit message: Finished Full-Bridge PCB, Fab Outputs
Parts:
- moved G*** 1.83 mm to (147.8, 64.0)
- moved TP35 1.70 mm to (165.3, 107.7)
- moved D3 0.94 mm to (161.1, 107.8)
- moved C50 0.11 mm to (125.6, 55.1)
- moved C32 0.10 mm to (128.4, 131.8)
- moved C52 0.09 mm to (123.5, 54.2)
- moved C51 0.09 mm to (121.2, 54.8)
Routing:
- net /Con_RDY_B_L: track 11.0 -> 108.5 mm, vias 1 -> 0
- net /Con_EN_B_L: track 11.1 -> 106.9 mm, vias 1 -> 0
- net /Con_RDY_B_H: track 11.5 -> 107.0 mm, vias 1 -> 2
- net /Con_FLT_B_L: track 11.2 -> 105.5 mm, vias 1 -> 0
- net /Con_FLT_B_H: track 11.3 -> 98.7 mm, vias 1 -> 2
- net /Con_EN_B_H: track 11.1 -> 89.5 mm, vias 1 -> 2
- net /Full-Bridge/Leg_A_Power_Stage/LegA_LS_Gate: track 44.8 -> 44.3 mm
